File: cp2102-atmega.sch (KiCad schematic (older format))
At the start: 20 parts

Commit message: Need yet to add the AVR programming connector and the RF filters
Parts:
- removed D? (x2): PESD5V0S1BB,115, Diodes_SMD:D_SOD-523, symbol nxp:TVS-2-pin
- added D? (x2): ESD8472MUT5G, on_semi:ONSEMI_0201_DSN2_153AF, symbol nxp:TVS-2-pin
Connections:
- net labels added: BYP_LNA1, BYP_LNA1_N, BYP_LNA2, BYP_LNA2_N, SWA_V1, SWA_V2, SWA_V3, SWB_V1, SWB_V2, SWB_V3
- wire segments 84 -> 94
Other:
- note added: "NEED TO ADD SPI PROGRAMMING CONNECTOR"
Changed lines of the file:
@@
 	2200 5550 2200 5600
-$Comp
-L nxp:TVS-2-pin D?
-U 1 1 5B7B78B3
-P 2850 5650
-F 0 "D?" H 2928 5703 60  0000 L CNN
-F 1 "PESD5V0S1BB,115" V 2700 5200 60  0000 L CNN
-F 2 "Diodes_SMD:D_SOD-523" H 2850 5650 60  0001 C CNN
-F 3 "https://assets.nexperia.com/documents/data-sheet/PESD5V0S1BA_BB_BL.pdf" H 2850 5650 60  0001 C CNN
-F 4 "Nexperia" H 2850 5650 50  0001 C CNN "Manufacturer"
-F 5 "PESD5V0S1BB,115" H 2850 5650 50  0001 C CNN "Part Number"
-F 6 "SOD-523" H 2850 5650 50  0001 C CNN "Package"
-F 7 "TVS DIODE 5V 14V SOD523" H 2850 5650 50  0001 C CNN "Description"
-	1    2850 5650
-	1    0    0    -1
-$EndComp
-$Comp
-L nxp:TVS-2-pin D?
-U 1 1 5B7B7C8D
-P 3300 5650
-F 0 "D?" H 3378 5703 60  0000 L CNN
-F 1 "PESD5V0S1BB,115" V 3150 5200 60  0000 L CNN
-F 2 "Diodes_SMD:D_SOD-523" H 3300 5650 60  0001 C CNN
-F 3 "https://assets.nexperia.com/documents/data-sheet/PESD5V0S1BA_BB_BL.pdf" H 3300 5650 60  0001 C CNN
-F 4 "Nexperia" H 3300 5650 50  0001 C CNN "Manufacturer"
-F 5 "PESD5V0S1BB,115" H 3300 5650 50  0001 C CNN "Part Number"
-F 6 "SOD-523" H 3300 5650 50  0001 C CNN "Package"
-F 7 "TVS DIODE 5V 14V SOD523" H 3300 5650 50  0001 C CNN "Description"
-	1    3300 5650
-	1    0    0    -1
-$EndComp
 $Comp
 L power:GND #PWR?
@@
 NoConn ~ 6100 4200
 NoConn ~ 6100 4100
+$Comp
+L nxp:TVS-2-pin D?
+U 1 1 5B92C2E9
+P 2850 5650
+AR Path="/5B782859/5B92C2E9" Ref="D?"  Part="1"
+AR Path="/5B7DAEA8/5B92C2E9" Ref="D?"  Part="1"
+F 0 "D?" H 2928 5703 60  0000 L CNN
+F 1 "ESD8472MUT5G" V 2700 5200 60  0000 L CNN
+F 2 "on_semi:ONSEMI_0201_DSN2_153AF" H 2850 5650 60  0001 C CNN
+F 3 "http://www.onsemi.com/pub/Collateral/ESD8472-D.PDF" H 2850 5650 60  0001 C CNN
+F 4 "ON Semiconductor" H 2850 5650 50  0001 C CNN "Manufacturer"
+F 5 "ESD8472MUT5G" H 2850 5650 50  0001 C CNN "Part Number"
+F 6 "0201 (0603 Metric)" H 2850 5650 50  0001 C CNN "Package"
+F 7 "TVS DIODE 5.3V 14V 2X3DFN" H 2850 5650 50  0001 C CNN "Description"
+	1    2850 5650
+	1    0    0    -1
+$EndComp
+$Comp
+L nxp:TVS-2-pin D?
+U 1 1 5B92E2C8
+P 3300 5650
+AR Path="/5B782859/5B92E2C8" Ref="D?"  Part="1"
+AR Path="/5B7DAEA8/5B92E2C8" Ref="D?"  Part="1"
+F 0 "D?" H 3378 5703 60  0000 L CNN
+F 1 "ESD8472MUT5G" V 3150 5200 60  0000 L CNN
+F 2 "on_semi:ONSEMI_0201_DSN2_153AF" H 3300 5650 60  0001 C CNN
+F 3 "http://www.onsemi.com/pub/Collateral/ESD8472-D.PDF" H 3300 5650 60  0001 C CNN
+F 4 "ON Semiconductor" H 3300 5650 50  0001 C CNN "Manufacturer"
+F 5 "ESD8472MUT5G" H 3300 5650 50  0001 C CNN "Part Number"
+F 6 "0201 (0603 Metric)" H 3300 5650 50  0001 C CNN "Package"
+F 7 "TVS DIODE 5.3V 14V 2X3DFN" H 3300 5650 50  0001 C CNN "Description"
+	1    3300 5650
+	1    0    0    -1
+$EndComp
+Text HLabel 8350 2700 0    50   Output ~ 0
+BYP_LNA1
+Text HLabel 8350 2800 0    50   Output ~ 0
+BYP_LNA1_N
+Text HLabel 8350 2900 0    50   Output ~ 0
+BYP_LNA2
+Text HLabel 8350 3000 0    50   Output ~ 0
+BYP_LNA2_N
+Text HLabel 8450 4600 0    50   Output ~ 0
+SWA_V1
+Text HLabel 8450 4700 0    50   Output ~ 0
+SWA_V2
+Text HLabel 8450 4800 0    50   Output ~ 0
+SWA_V3
+Text HLabel 8450 4900 0    50   Output ~ 0
+SWB_V1
+Text HLabel 8450 5000 0    50   Output ~ 0
+SWB_V2
+Text HLabel 8450 5100 0    50   Output ~ 0
+SWB_V3
+Wire Wire Line
+	8450 4600 8950 4600
+Wire Wire Line
+	8450 4700 8950 4700
+Wire Wire Line
+	8450 4800 8950 4800
+Wire Wire Line
+	8450 4900 8950 4900
+Wire Wire Line
+	8450 5000 8950 5000
+Wire Wire Line
+	8450 5100 8950 5100
+Wire Wire Line
+	8350 2700 8950 2700
+Wire Wire Line
+	8350 2800 8950 2800
+Wire Wire Line
+	8350 2900 8950 2900
+Wire Wire Line
+	8350 3000 8950 3000
+Text Notes 3200 3000 0    100  ~ 20
+NEED TO ADD SPI PROGRAMMING CONNECTOR
 $EndSCHEMATC

Commit message: Schematic complete. Ready for review.
Parts:
- added C1, C5: 1uF, Capacitors_SMD:C_0402, symbol Device:C
- added C10, C15, C3: 100nF, Capacitors_SMD:C_0402, symbol Device:C
- added D4: PESD12VS1UB,115, Diodes_SMD:D_SOD-523, symbol Diode:1.5KExxA
- added J2: Conn_02x03_Odd_Even, amphenol:FRAMATOME_67997-206HLF, symbol Connector_Generic:Conn_02x03_Odd_Even
- added R4: 10K, Resistors_SMD:R_0402, symbol Device:R
- added R5: 0, Resistors_SMD:R_0402, symbol Device:R
- added U1: TPS73233DBVR, Package_TO_SOT_SMD:TSOT-23-5, symbol Regulator_Linear:ADP7142AUZJ
- gave numbers to parts that had none: 20
Connections:
- net labels added: +3.3V, +3.3VA, MISO, MOSI, SCK, VCC, ~RESET
- net labels removed: +3V3_DIG
- wire segments 94 -> 131
- no-connect marks 13 -> 22
Other:
- note added: "AVR\nprogramming"
- note added: "analog\nsupply"
- note added: "digital\nsupply"
- note removed: "NEED TO ADD SPI PROGRAMMING CONNECTOR"
- moved on the sheet: J1

Commit message: More updates. Added LED to AVR to help with bring up and debug.
Parts:
- added D?: SML-LX0402SUGC-TR, LEDs:LED_0402, symbol Device:LED
- added R?: 1K, Resistors_SMD:R_0402, symbol Device:R
Connections:
- net labels added: LED_GRN
- wire segments 131 -> 135
- no-connect marks 22 -> 21
Changed lines of the file:
@@
 NoConn ~ 10150 2900
 NoConn ~ 10150 3000
-NoConn ~ 8950 2700
 NoConn ~ 8950 2800
 NoConn ~ 8950 2900
@@
 Wire Wire Line
 	1600 6050 2650 6050
+$Comp
+L Device:LED D?
+U 1 1 5BF7029D
+P 7150 3400
+F 0 "D?" V 7188 3283 50  0000 R CNN
+F 1 "SML-LX0402SUGC-TR" V 7097 3283 50  0000 R CNN
+F 2 "LEDs:LED_0402" H 7150 3400 50  0001 C CNN
+F 3 "https://www.lumex.com/content/files/ProductAttachment/SML-LX0402SUGC-TR.pdf" H 7150 3400 50  0001 C CNN
+F 4 "Lumex" H 7150 3400 50  0001 C CNN "Manufacturer"
+F 5 "SML-LX0402SUGC-TR" H 7150 3400 50  0001 C CNN "Part Number"
+F 6 "0402" H 7150 3400 50  0001 C CNN "Package"
+F 7 "LED GREEN CLEAR SMD" H 7150 3400 50  0001 C CNN "Description"
+	1    7150 3400
+	0    -1   -1   0
+$EndComp
+$Comp
+L Device:R R?
+U 1 1 5BF704B7
+P 7150 3050
+F 0 "R?" H 7220 3096 50  0000 L CNN
+F 1 "1K" V 7150 3000 50  0000 L CNN
+F 2 "Resistors_SMD:R_0402" V 7080 3050 50  0001 C CNN
+F 3 "~" H 7150 3050 50  0001 C CNN
+F 4 "Panasonic" H 7150 3050 50  0001 C CNN "Manufacturer"
+F 5 "ERJ-2RKF1001X" H 7150 3050 50  0001 C CNN "Part Number"
+F 6 "0402" H 7150 3050 50  0001 C CNN "Package"
+F 7 "RES SMD 1K OHM 1% 1/10W 0402" H 7150 3050 50  0001 C CNN "Description"
+F 8 "RCA04021K00FKEDHP" H 7150 3050 50  0001 C CNN "Alternate Part Number"
+	1    7150 3050
+	1    0    0    -1
+$EndComp
+Wire Wire Line
+	7150 3200 7150 3250
+$Comp
+L power:GND #PWR?
+U 1 1 5BF7F1BE
+P 7150 3600
+F 0 "#PWR?" H 7150 3350 50  0001 C CNN
+F 1 "GND" H 7155 3427 50  0000 C CNN
+F 2 "" H 7150 3600 50  0001 C CNN
+F 3 "" H 7150 3600 50  0001 C CNN
+	1    7150 3600
+	1    0    0    -1
+$EndComp
+Wire Wire Line
+	7150 3550 7150 3600
+Wire Wire Line
+	8950 2700 7150 2700
+Wire Wire Line
+	7150 2700 7150 2900
+Text Label 8450 2700 0    50   ~ 0
+LED_GRN
 $EndSCHEMATC

Commit message: Started parts placement and fixed some RF routing to accomodate layout
Parts:
- removed C14: 100nF, Capacitors_SMD:C_0402, symbol Device:C
- U1, U2: footprint Package_TO_SOT_SMD:TSOT-23-5 -> TO_SOT_Packages_SMD:SOT-23-5
- U3: footprint Package_DFN_QFN:QFN-24-1EP_4x4mm_P0.5mm_EP2.6x2.6mm -> Housings_DFN_QFN:QFN-24-1EP_4x4mm_Pitch0.5mm
- U4: footprint Package_DFN_QFN:QFN-32-1EP_5x5mm_P0.5mm_EP3.1x3.1mm -> Housings_DFN_QFN:QFN-32-1EP_5x5mm_Pitch0.5mm
- gave numbers to parts that had none: 2
Connections:
- wire segments 135 -> 132
Changed lines of the file:
@@
 F 0 "U4" H 8950 2650 50  0000 C CNN
 F 1 "ATmega328P-MU" H 8700 2550 50  0000 C CNN
-F 2 "Package_DFN_QFN:QFN-32-1EP_5x5mm_P0.5mm_EP3.1x3.1mm" H 9550 3900 50  0001 C CIN
+F 2 "Housings_DFN_QFN:QFN-32-1EP_5x5mm_Pitch0.5mm" H 9550 3900 50  0001 C CIN
 F 3 "http://ww1.microchip.com/downloads/en/DeviceDoc/ATmega328_P%20AVR%20MCU%20with%20picoPower%20Technology%20Data%20Sheet%2040001984A.pdf" H 9550 3900 50  0001 C CNN
 F 4 "Microchip Technology" H 9550 3900 50  0001 C CNN "Manufacturer"
@@
 F 0 "U3" H 4100 6650 50  0000 C CNN
 F 1 "CP2102N-A01-GQFN24" H 5000 6650 50  0000 C CNN
-F 2 "Package_DFN_QFN:QFN-24-1EP_4x4mm_P0.5mm_EP2.6x2.6mm" H 4950 5050 50  0001 L CNN
+F 2 "Housings_DFN_QFN:QFN-24-1EP_4x4mm_Pitch0.5mm" H 4950 5050 50  0001 L CNN
 F 3 "http://www.silabs.com/support%20documents/technicaldocs/cp2102n-datasheet.pdf" H 4550 4800 50  0001 C CNN
 F 4 "Silicon Labs" H 4500 5850 50  0001 C CNN "Manufacturer"
@@
 	0    1    1    0
 $EndComp
-$Comp
-L Device:C C14
-U 1 1 5B791580
-P 10100 2000
-F 0 "C14" V 9950 2000 50  0000 L CNN
-F 1 "100nF" V 10250 1900 50  0000 L CNN
-F 2 "Capacitors_SMD:C_0402" H 10138 1850 50  0001 C CNN
-F 3 "~" H 10100 2000 50  0001 C CNN
-F 4 "CL05A104MP5NNNC" H 10100 2000 50  0001 C CNN "Part Number"
-F 5 "0402" H 10100 2000 50  0001 C CNN "Package"
-F 6 "CAP CER 0.1UF 10V X5R 0402" H 10100 2000 50  0001 C CNN "Description"
-F 7 "6.3V or greater" H 10100 2000 50  0001 C CNN "Notes"
-F 8 "GRM022R60J104ME15L" H 10100 2000 50  0001 C CNN "Alternate Part Number"
-	1    10100 2000
-	0    1    1    0
-$EndComp
 Wire Wire Line
 	9100 2000 9450 2000
@@
 Wire Wire Line
 	9450 2250 9450 2400
-Wire Wire Line
-	9950 2000 9550 2000
 Wire Wire Line
 	9550 2000 9550 2250
@@
 $EndComp
 Wire Wire Line
-	10250 2000 10300 2000
-Wire Wire Line
-	10300 2000 10300 2250
-Wire Wire Line
 	10000 2250 10300 2250
-Connection ~ 10300 2250
 Wire Wire Line
 	10300 2250 10300 2300
@@
 	9450 2000 9500 2000
 Connection ~ 9450 2000
-Connection ~ 9550 2000
 Connection ~ 9500 2000
 Wire Wire Line
@@
 F 0 "U2" H 2250 1817 50  0000 C CNN
 F 1 "TPS73233DBVR" H 2250 1726 50  0000 C CNN
-F 2 "Package_TO_SOT_SMD:TSOT-23-5" H 2250 1050 50  0001 C CIN
+F 2 "TO_SOT_Packages_SMD:SOT-23-5" H 2250 1050 50  0001 C CIN
 F 3 "http://www.ti.com/lit/ds/symlink/tps732.pdf" H 2250 950 50  0001 C CNN
 F 4 "Texas Instruments" H 2250 1450 50  0001 C CNN "Manufacturer"
@@
 F 0 "U1" H 2200 3217 50  0000 C CNN
 F 1 "TPS73233DBVR" H 2200 3126 50  0000 C CNN
-F 2 "Package_TO_SOT_SMD:TSOT-23-5" H 2200 2450 50  0001 C CIN
+F 2 "TO_SOT_Packages_SMD:SOT-23-5" H 2200 2450 50  0001 C CIN
 F 3 "http://www.ti.com/lit/ds/symlink/tps732.pdf" H 2200 2350 50  0001 C CNN
 F 4 "Texas Instruments" H 2200 2850 50  0001 C CNN "Manufacturer"
@@
 	1600 6050 2650 6050
 $Comp
-L Device:LED D?
+L Device:LED D9
 U 1 1 5BF7029D
 P 7150 3400
-F 0 "D?" V 7188 3283 50  0000 R CNN
+F 0 "D9" V 7188 3283 50  0000 R CNN
 F 1 "SML-LX0402SUGC-TR" V 7097 3283 50  0000 R CNN
 F 2 "LEDs:LED_0402" H 7150 3400 50  0001 C CNN
@@
 $EndComp
 $Comp
-L Device:R R?
+L Device:R R20
 U 1 1 5BF704B7
 P 7150 3050
-F 0 "R?" H 7220 3096 50  0000 L CNN
+F 0 "R20" H 7220 3096 50  0000 L CNN
 F 1 "1K" V 7150 3000 50  0000 L CNN
 F 2 "Resistors_SMD:R_0402" V 7080 3050 50  0001 C CNN
@@
 	7150 3200 7150 3250
 $Comp
-L power:GND #PWR?
+L power:GND #PWR0122
 U 1 1 5BF7F1BE
 P 7150 3600
-F 0 "#PWR?" H 7150 3350 50  0001 C CNN
+F 0 "#PWR0122" H 7150 3350 50  0001 C CNN
 F 1 "GND" H 7155 3427 50  0000 C CNN
 F 2 "" H 7150 3600 50  0001 C CNN
