File: rf_section.sch (KiCad schematic (older format))
At the start: 58 parts

Commit message: Schematic complete. Ready for review.
Parts:
- removed C? (x2): 1uF, Capacitors_SMD:C_0402, symbol Device:C
- removed C?: 100nF, Capacitors_SMD:C_0402, symbol Device:C
- removed U?: TPS73233DBVR, Package_TO_SOT_SMD:TSOT-23-5, symbol Regulator_Linear:ADP7142AUZJ
- added FL1: TA1090EC, saw_filters:SAW_3.8X3.8MM, symbol murata:SAW_3X3mm
- added FL2: SF2098E, saw_filters:SAW_3X3mm, symbol murata:SAW_3X3mm
- added FL3: SF2250E, saw_filters:SAW_3X3mm, symbol murata:SAW_3X3mm
- gave numbers to parts that had none: 54
Connections:
- net labels removed: VBUS
- wire segments 219 -> 237

Commit message: More updates. Added LED to AVR to help with bring up and debug.
Other:
- note added: "V1 V2 V3 RF\n0 0 0 1\n0 0 1 2\n0 1 0 3\n0 1 1 4\n1 0 0 ISO\n1 0 1 50 Ohm\n1 1 1 SHDN"
Changed lines of the file:
@@
 Wire Wire Line
 	1450 3750 1450 4900
+Text Notes 9550 5800 0    50   ~ 10
+V1      V2      V3     RF\n0        0       0      1\n0        0       1      2\n0        1       0      3\n0        1       1      4\n1        0       0      ISO\n1        0       1      50 Ohm\n1        1       1      SHDN
 $EndSCHEMATC

Commit message: Started parts placement and fixed some RF routing to accomodate layout
Connections:
- wire segments 237 -> 236
Other:
- note added: "BAND SWA_V1 SWA_V2 SWA_V3 SWB_V1 SWB_V2 SWB_V3\nFL1 0 1 0 0 1 1\nFL2 0 0 1 0 0 0\nFL3 0 0 0 0 0 1\nEXT 0 1 1 0 1 0"
