File: rf-section.sch (KiCad schematic (older format))
At the start: 57 parts, among them J3 SMA-J-P-H-ST-EM1, J4 SMA-J-P-H-ST-EM1, J5 SMA-J-P-H-ST-EM1, J6 SMA-J-P-H-ST-EM1, U10 SPF5122Z, U11 SKY13414-485LF, U12 SKY13351-378LF, U5 SKY13414-485LF, U6 SKY13351-378LF, U7 SPF5122Z, U8 SKY13351-378LF, U9 SKY13351-378LF

Commit message: Changed design to be a pi-hat
Parts:
- renumbered C16 to C15, C17 to C16, C18 to C17, C20 to C18, C21 to C19, C19 to C20, C23 to C21, C24 to C23, C25 to C24, C26 to C25, C30 to C26, C32 to C28, C35 to C29, C28 to C30, C29 to C31, C31 to C32, C36 to C35, C37 to C36, D5 to D6, D6 to D7, D7 to D8, D8 to D9, FL2 to FL1, FL3 to FL2, FL1 to FL3, J3 to J4, J4 to J5, J5 to J7, J6 to J8, R6 to R12, R7 to R13, R8 to R14, R9 to R15, R10 to R16, R11 to R17, R12 to R18, R13 to R19, R14 to R20, R15 to R21, R16 to R22, R17 to R25, R18 to R26, R19 to R27, U9 to U10, U10 to U11, U11 to U12, U12 to U13, U5 to U6, U6 to U7, U7 to U8, U8 to U9

Commit message: Almost all 3D models have been added. Rough parts placement complete.
Parts:
- removed J4, J5, J7, J8: SMA-J-P-H-ST-EM1, samtec:SMA-J-P-H-ST-EM1, symbol samtec:SMA-J-P-H-ST-EM1
- added J4, J5, J7, J8: 619540-1, project_footprints:619540-1, symbol rf_connectors:RF-GND1
- C15, C16, C17, C18, C19, C20, C21, C22, C23, C24, C25, C26, C27, C28, C29, C30, C31, C32, C33, C34, C35, C36: footprint Capacitors_SMD:C_0402 -> project_footprints:C_0402
- D6, D7, D8, D9: footprint on_semi:ONSEMI_0201_DSN2_153AF -> project_footprints:ONSEMI_0201_DSN2_153AF
- FL1, FL2: footprint saw_filters:SAW_3X3mm -> project_footprints:SAW_3X3mm
- FL3: footprint saw_filters:SAW_3.8X3.8MM -> project_footprints:SAW_3.8X3.8MM
- L1, L2: footprint Inductors_SMD:L_0603 -> project_footprints:L_0603
- R12, R13, R14, R15, R16, R17, R18, R19, R20, R21, R22, R25, R26, R27: footprint Resistors_SMD:R_0402 -> project_footprints:R_0402
- U10, U13, U7, U9: footprint skyworks:SKY_QFN6_1x1mm -> project_footprints:SKY_QFN6_1x1mm
- U11, U8: footprint qorvo:DFN-8 -> project_footprints:DFN-8
- U12, U6: footprint skyworks:QFN45P200X200X55-15N -> project_footprints:QFN45P200X200X55-15N
Connections:
- wire segments 236 -> 243

Commit message: Trimmed unnecessary parts from the Pi power circuitry. Now the Pi 5V is diode or'd with VBUS from the USB
Parts:
- removed C24: 100nF, project_footprints:C_0402, symbol Device:C
- removed C25, C27, C30, C31, C33, C36: 100pF, project_footprints:C_0402, symbol Device:C
- removed R19, R20, R26, R27: 100, project_footprints:R_0402, symbol Device:R
- removed U10, U13, U7, U9: SKY13351-378LF, project_footprints:SKY_QFN6_1x1mm, symbol skyworks:SKY13351-378LF
- removed U11, U8: SPF5122Z, project_footprints:DFN-8, symbol qorvo:SPF5122Z
- added C12: 100pF, project_footprints:C_0402, symbol Device:C
- added L3, L4: 12nH, project_footprints:LQW15A, symbol Device:L
- added M1, M2: 2118706-2, project_footprints:2118706-2, symbol te_connectivity:SHEILD8
- added U7, U8: GRF4042, project_footprints:QFN-12_EP_2x2_Pitch0.5mm, symbol guerilla_rf:GRF4042
- C15: value 100pF -> 100nF; Alternate Part Number 500X07N101MV4T -> GRM022R60J104ME15L; Description CAP CER 100PF 25V C0G/NP0 01005 -> CAP CER 0.1UF 10V X5R 0402; Manufacturer Murata -> (none); Notes (none) -> 6.3V or greater; Part Number GRM0225C1E101GA02L -> CL05A104MP5NNNC
- FL2: Description FILTER SAW 1.615GHZ 6SMD -> FILTER SAW FC=1615MHZ BW=20MHz 6SMD
- FL3: value TA1090EC -> SF2275E; footprint project_footprints:SAW_3.8X3.8MM -> project_footprints:SAW_3X3mm; Description FILTER SAW 1090MHz -> FILTER SAW FC=1542.5MHZ BW=35MHz; Manufacturer TAI-SAW -> Murata; Package SAW 3.8x3.8mm -> SAW 3x3mm; Part Number TA1090EC -> SF2275E
- L1, L2: value 150nH -> 12nH; footprint project_footprints:L_0603 -> project_footprints:LQW15A; Description FIXED IND 150NH 300MA 1.4 OHM -> FIXED IND 12NH 1.24A 93 MOHM; Manufacturer Johanson Technology -> Murata; Package 0603 -> 0402; Part Number L-14CR15JV4T -> LQW15AN12NJ8ZD
- R13, R18: value 100 -> 374; Alternate Part Number RT0402FRE071KL -> RC0402FR-07374RL; Description RES SMD 1K OHM 1% 1/10W 0402 -> RES SMD 374 OHM 1% 1/10W 0402; Part Number ERJ-2RKF1001X -> ERJ-2RKF3740X
Connections:
- net labels removed: BYP_LNA1_N, BYP_LNA2_N
- wire segments 243 -> 244

Commit message: Can now power via: 1. USB 2. R-Pi 3. Bias TEE
Parts:
- added C24: 1uF, project_footprints:C_0402, symbol Device:C
- added L5: 1uH, murata:INDC2520X100, symbol pspice:INDUCTOR
Connections:
- net labels added: +5VP
- wire segments 244 -> 250
Changed lines of the file:
@@
 L power:GND #PWR057
 U 1 1 5B95A466
-P 4650 7000
-F 0 "#PWR057" H 4650 6750 50  0001 C CNN
-F 1 "GND" H 4655 6827 50  0000 C CNN
-F 2 "" H 4650 7000 50  0001 C CNN
-F 3 "" H 4650 7000 50  0001 C CNN
-	1    4650 7000
+P 6400 7000
+F 0 "#PWR057" H 6400 6750 50  0001 C CNN
+F 1 "GND" H 6405 6827 50  0000 C CNN
+F 2 "" H 6400 7000 50  0001 C CNN
+F 3 "" H 6400 7000 50  0001 C CNN
+	1    6400 7000
 	-1   0    0    -1
 $EndComp
@@
 L nxp:TVS-2-pin D?
 U 1 1 5B9767C9
-P 4250 6900
+P 6000 6900
 AR Path="/5B782859/5B9767C9" Ref="D?"  Part="1"
 AR Path="/5B7DAEA8/5B9767C9" Ref="D?"  Part="1"
 AR Path="/5C1B2C8B/5B9767C9" Ref="D8"  Part="1"
-F 0 "D8" V 4150 6850 60  0000 L CNN
-F 1 "ESD8472MUT5G" V 4350 6550 60  0000 L CNN
-F 2 "project_footprints:ONSEMI_0201_DSN2_153AF" H 4250 6900 60  0001 C CNN
-F 3 "http://www.onsemi.com/pub/Collateral/ESD8472-D.PDF" H 4250 6900 60  0001 C CNN
-F 4 "ON Semiconductor" H 4250 6900 50  0001 C CNN "Manufacturer"
-F 5 "ESD8472MUT5G" H 4250 6900 50  0001 C CNN "Part Number"
-F 6 "0201 (0603 Metric)" H 4250 6900 50  0001 C CNN "Package"
-F 7 "TVS DIODE 5.3V 14V 2X3DFN" H 4250 6900 50  0001 C CNN "Description"
-	1    4250 6900
+F 0 "D8" V 5900 6850 60  0000 L CNN
+F 1 "ESD8472MUT5G" V 6100 6550 60  0000 L CNN
+F 2 "project_footprints:ONSEMI_0201_DSN2_153AF" H 6000 6900 60  0001 C CNN
+F 3 "http://www.onsemi.com/pub/Collateral/ESD8472-D.PDF" H 6000 6900 60  0001 C CNN
+F 4 "ON Semiconductor" H 6000 6900 50  0001 C CNN "Manufacturer"
+F 5 "ESD8472MUT5G" H 6000 6900 50  0001 C CNN "Part Number"
+F 6 "0201 (0603 Metric)" H 6000 6900 50  0001 C CNN "Package"
+F 7 "TVS DIODE 5.3V 14V 2X3DFN" H 6000 6900 50  0001 C CNN "Description"
+	1    6000 6900
 	0    1    1    0
 $EndComp
@@
 	1950 1950 1350 1950
 Wire Wire Line
-	4650 6750 4050 6750
-Connection ~ 4050 6750
+	6400 6750 5800 6750
+Connection ~ 5800 6750
 Wire Wire Line
 	3700 1750 4150 1750
@@
 	4150 1950 4150 1750
 Connection ~ 4150 1750
-Wire Wire Line
-	4150 1750 4200 1750
 $Comp
 L Device:R R?
@@
 Text Notes 9550 5800 0    50   ~ 10
 V1      V2      V3     RF\n0        0       0      1\n0        0       1      2\n0        1       0      3\n0        1       1      4\n1        0       0      ISO\n1        0       1      50 Ohm\n1        1       1      SHDN
-Text Notes 5500 6350 0    50   ~ 10
+Text Notes 6450 5800 0    50   ~ 10
 BAND    SWA_V1    SWA_V2    SWA_V3     SWB_V1     SWB_V2    SWB_V3\nFL1         0         1          0          0            1           1\nFL2         0         0          1          0            0           0\nFL3         0         0          0          0            0           1\nEXT         0         1          1          0            1           0
 Wire Wire Line
@@
 L rf_connectors:RF-GND1 J7
 U 1 1 5B86BC5C
-P 4850 6750
-F 0 "J7" H 4779 6986 50  0000 C CNN
-F 1 "619540-1" H 4779 6895 50  0000 C CNN
-F 2 "project_footprints:619540-1" H 4850 6750 50  0001 C CNN
-F 3 "" H 4850 6750 50  0001 C CNN
-F 4 "TE Connectivity" H 4850 6750 50  0001 C CNN "Manufacturer"
-F 5 "619540-1" H 4850 6750 50  0001 C CNN "Part Number"
-F 6 "SMA THRU RA" H 4850 6750 50  0001 C CNN "Package"
-F 7 "SMA Connector Jack, Female Socket 50 Ohm Through Hole, Right Angle Solder" H 4850 6750 50  0001 C CNN "Description"
-	1    4850 6750
-	1    0    0    -1
-$EndComp
-Wire Wire Line
-	4050 6900 4050 6750
-Wire Wire Line
-	4450 6900 4650 6900
-Wire Wire Line
-	4650 6900 4650 7000
-Connection ~ 4650 6900
-Wire Wire Line
-	4650 6900 4850 6900
+P 6600 6750
+F 0 "J7" H 6529 6986 50  0000 C CNN
+F 1 "619540-1" H 6529 6895 50  0000 C CNN
+F 2 "project_footprints:619540-1" H 6600 6750 50  0001 C CNN
+F 3 "" H 6600 6750 50  0001 C CNN
+F 4 "TE Connectivity" H 6600 6750 50  0001 C CNN "Manufacturer"
+F 5 "619540-1" H 6600 6750 50  0001 C CNN "Part Number"
+F 6 "SMA THRU RA" H 6600 6750 50  0001 C CNN "Package"
+F 7 "SMA Connector Jack, Female Socket 50 Ohm Through Hole, Right Angle Solder" H 6600 6750 50  0001 C CNN "Description"
+	1    6600 6750
+	1    0    0    -1
+$EndComp
+Wire Wire Line
+	5800 6900 5800 6750
+Wire Wire Line
+	6200 6900 6400 6900
+Wire Wire Line
+	6400 6900 6400 7000
+Connection ~ 6400 6900
+Wire Wire Line
+	6400 6900 6600 6900
 Wire Wire Line
 	2200 4200 2750 4200
@@
 	0    -1   -1   0
 $EndComp
-Wire Wire Line
-	3900 6750 4050 6750
 $Comp
 L te_connectivity:SHEILD8 M2
@@
 Wire Wire Line
 	4600 5850 4600 5950
+Wire Wire Line
+	4150 1750 4200 1750
+Wire Wire Line
+	3900 6750 5300 6750
+$Comp
+L pspice:INDUCTOR L5
+U 1 1 5B9C6C97
+P 5300 6400
+F 0 "L5" V 5254 6478 50  0000 L CNN
+F 1 "1uH" V 5345 6478 50  0000 L CNN
+F 2 "murata:INDC2520X100" H 5300 6400 50  0001 C CNN
+F 3 "https://search.murata.co.jp/Ceramy/image/img/P02/JELF243A-0085.pdf" H 5300 6400 50  0001 C CNN
+F 4 "Murata" H 5300 6400 50  0001 C CNN "Manufacturer"
+F 5 "LQW2UAS1R0J00L" H 5300 6400 50  0001 C CNN "Part Number"
+F 6 "1008 (2520 Metric)" H 5300 6400 50  0001 C CNN "Package"
+F 7 "1µH Unshielded Wirewound Inductor 370mA 1.75 Ohm Max 1008 (2520 Metric)" H 5300 6400 50  0001 C CNN "Description"
+	1    5300 6400
+	0    1    1    0
+$EndComp
+Wire Wire Line
+	5300 6650 5300 6750
+Connection ~ 5300 6750
+Wire Wire Line
+	5300 6750 5800 6750
+$Comp
+L Device:C C?
+U 1 1 5B9D97E3
+P 5700 5950
+AR Path="/5C1B036A/5B9D97E3" Ref="C?"  Part="1"
+AR Path="/5B9D97E3" Ref="C?"  Part="1"
+AR Path="/5C1B2C8B/5B9D97E3" Ref="C24"  Part="1"
+F 0 "C24" H 5700 6050 50  0000 L CNN
+F 1 "1uF" H 5700 5850 50  0000 L CNN
+F 2 "project_footprints:C_0402" H 5738 5800 50  0001 C CNN
+F 3 "~" H 5700 5950 50  0001 C CNN
+F 4 "Murata" H 5700 5950 50  0001 C CNN "Manufacturer"
+F 5 "GRM153R60J105ME95D" H 5700 5950 50  0001 C CNN "Part Number"
+F 6 "0402" H 5700 5950 50  0001 C CNN "Package"
+F 7 "CAP 1UF 6.3V X5R 0402" H 5700 5950 50  0001 C CNN "Description"
+F 8 "6.3V or greater" H 5700 5950 50  0001 C CNN "Notes"
+F 9 "CL05A105MQ3LNNH" H 5700 5950 50  0001 C CNN "Alternate Part Number"
+	1    5700 5950
+	1    0    0    -1
+$EndComp
+$Comp
+L power:GND #PWR070
+U 1 1 5B9EA2AF
+P 5700 6150
+F 0 "#PWR070" H 5700 5900 50  0001 C CNN
+F 1 "GND" H 5705 5977 50  0000 C CNN
+F 2 "" H 5700 6150 50  0001 C CNN
+F 3 "" H 5700 6150 50  0001 C CNN
+	1    5700 6150
+	-1   0    0    -1
+$EndComp
+Wire Wire Line
+	5700 6100 5700 6150
+Wire Wire Line
+	5700 5800 5300 5800
+Wire Wire Line
+	5300 5800 5300 6150
+$Comp
+L power:+5VP #PWR?
+U 1 1 5BA100FD
+P 5300 5700
+AR Path="/5BA100FD" Ref="#PWR?"  Part="1"
+AR Path="/5C1B2C8B/5BA100FD" Ref="#PWR069"  Part="1"
+F 0 "#PWR069" H 5300 5550 50  0001 C CNN
+F 1 "+5VP" H 5315 5873 50  0000 C CNN
+F 2 "" H 5300 5700 50  0001 C CNN
+F 3 "" H 5300 5700 50  0001 C CNN
+	1    5300 5700
+	1    0    0    -1
+$EndComp
+Wire Wire Line
+	5300 5700 5300 5800
+Connection ~ 5300 5800
 $EndSCHEMATC

Commit message: Finally have the stackup
Parts:
- removed J4, J5, J7, J8: 619540-1, project_footprints:619540-1, symbol rf_connectors:RF-GND1
- added J4, J5, J7, J8: SMA-J-P-H-ST-EM1, samtec:SMA-J-P-H-ST-EM1, symbol samtec:SMA-J-P-H-ST-EM1
- U7, U8: value GRF4042 -> GRF4142; Part Number GRF4042 -> GRF4142
Connections:
- wire segments 250 -> 249

Commit message: I think the layout is ready for review
Parts:
- removed C21: 100pF, project_footprints:C_0402, symbol Device:C
- removed R13, R18: 374, project_footprints:R_0402, symbol Device:R
- removed U7, U8: GRF4142, project_footprints:QFN-12_EP_2x2_Pitch0.5mm, symbol guerilla_rf:GRF4042
- added C25, C31: 30pF, project_footprints:C_0402, symbol Device:C
- added C27, C33: DNF, project_footprints:C_0402, symbol Device:C
- added C30, C36: 1pF, project_footprints:C_0402, symbol Device:C
- added C37: 100pF, project_footprints:C_0402, symbol Device:C
- added L6: BLM15AG121SN1D, murata:FB_0402_NoSilk, symbol Device:Ferrite_Bead
- added U7, U8: GRF4142, guerilla_rf:DFN1.5MMX1.5MMX0.45MM-6, symbol guerilla_rf:GRF4142
- L1, L3: value 12nH -> 22nH; footprint project_footprints:LQW15A -> murata:L_0402; Alternate Part Number HK1608R15J-T -> MLG1005S22NJT000; Description FIXED IND 12NH 1.24A 93 MOHM -> FIXED IND 22NH 350MA 420 MOHM; Package 0402 -> L_0402; Part Number LQW15AN12NJ8ZD -> LQG15HS22NJ02D
- L2, L4: value 12nH -> 39nH; footprint project_footprints:LQW15A -> murata:L_0402; Alternate Part Number HK1608R15J-T -> MLK1005S39NJTD25; Description FIXED IND 12NH 1.24A 93 MOHM -> FIXED IND 39NH 300MA 650 MOHM; Package 0402 -> L_0402; Part Number LQW15AN12NJ8ZD -> LQG15HS39NJ02D
- R12, R17: value 100 -> 1.4K; Alternate Part Number RT0402FRE071KL -> RC0402FR-071K4L; Description RES SMD 1K OHM 1% 1/10W 0402 -> RES SMD 1.4K OHM 1% 1/10W 0402; Part Number ERJ-2RKF1001X -> ERJ-2RKF1401X
Connections:
- wire segments 249 -> 238

Commit message: Cleaned up BOM and added part numbers to the layout.
Parts:
- C15, C18, C32, C35: Manufacturer (none) -> Samsung
- J4, J5, J7, J8: Description (none) -> SMA Connector Jack, Female Socket 50 Ohm Board Edge, End La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; Field4 None -> (none); Field5 SMA-J-P-H-ST-EM1 -> (none); Field6 Good -> (none); Field7 2.95 USD -> (none); Field8 Samtec -> (none); Manufacturer (none) -> Samtec; Package (none) -> SMA_END_LAUNCH; Part Number (none) -> SMA-J-P-H-ST-EM1
- U7, U8: Description (none) -> RF Amplifier .1-3.8GHz GaAs Gain 16dB
Other:
- note added: "BAND SWA_V1 SWA_V2 SWA_V3 SWB_V1 SWB_V2 SWB_V3\nFL1 0 0 0 0 0 1\nFL2 0 1 0 0 1 1\nFL3 0 0 1 0 0 0\nEXT 0 1 1 0 1 0"
- note removed: "BAND SWA_V1 SWA_V2 SWA_V3 SWB_V1 SWB_V2 SWB_V3\nFL1 0 1 0 0 1 1\nFL2 0 0 1 0 0 0\nFL3 0 0 0 0 0 1\nEXT 0 1 1 0 1 0"
Changed lines of the file:
@@
 Title ""
 Date ""
-Rev ""
-Comp ""
+Rev "A"
+Comp "505-201"
 Comment1 ""
 Comment2 ""
@@
 F 7 "6.3V or greater" H 6950 1150 50  0001 C CNN "Notes"
 F 8 "GRM022R60J104ME15L" H 6950 1150 50  0001 C CNN "Alternate Part Number"
+F 9 "Samsung" H 0   0   50  0001 C CNN "Manufacturer"
 	1    6950 1150
 	0    1    1    0
@@
 F 7 "6.3V or greater" H 9800 3400 50  0001 C CNN "Notes"
 F 8 "GRM022R60J104ME15L" H 9800 3400 50  0001 C CNN "Alternate Part Number"
+F 9 "Samsung" H 0   0   50  0001 C CNN "Manufacturer"
 	1    9800 3400
 	0    1    1    0
@@
 F 7 "6.3V or greater" H 2400 3900 50  0001 C CNN "Notes"
 F 8 "GRM022R60J104ME15L" H 2400 3900 50  0001 C CNN "Alternate Part Number"
+F 9 "Samsung" H 0   0   50  0001 C CNN "Manufacturer"
 	1    2400 3900
 	0    1    1    0
@@
 V1      V2      V3     RF\n0        0       0      1\n0        0       1      2\n0        1       0      3\n0        1       1      4\n1        0       0      ISO\n1        0       1      50 Ohm\n1        1       1      SHDN
 Text Notes 6450 5800 0    50   ~ 10
-BAND    SWA_V1    SWA_V2    SWA_V3     SWB_V1     SWB_V2    SWB_V3\nFL1         0         1          0          0            1           1\nFL2         0         0          1          0            0           0\nFL3         0         0          0          0            0           1\nEXT         0         1          1          0            1           0
+BAND    SWA_V1    SWA_V2    SWA_V3     SWB_V1     SWB_V2    SWB_V3\nFL1         0         0          0          0            0           1\nFL2         0         1          0          0            1           1\nFL3         0         0          1          0            0           0\nEXT         0         1          1          0            1           0
 Wire Wire Line
 	7200 4750 9450 4750
@@
 F 7 "6.3V or greater" H 4150 6200 50  0001 C CNN "Notes"
 F 8 "GRM022R60J104ME15L" H 4150 6200 50  0001 C CNN "Alternate Part Number"
+F 9 "Samsung" H 0   0   50  0001 C CNN "Manufacturer"
 	1    4150 6200
 	0    1    1    0
@@
 F 2 "samtec:SMA-J-P-H-ST-EM1" H 950 1950 50  0001 L BNN
 F 3 "Connector SMA F 50Ohm Solder ST Edge Mount Gold Over Nickel Tray" H 950 1950 50  0001 L BNN
-F 4 "None" H 950 1950 50  0001 L BNN "Field4"
-F 5 "SMA-J-P-H-ST-EM1" H 950 1950 50  0001 L BNN "Field5"
-F 6 "Good" H 950 1950 50  0001 L BNN "Field6"
-F 7 "2.95 USD" H 950 1950 50  0001 L BNN "Field7"
-F 8 "Samtec" H 950 1950 50  0001 L BNN "Field8"
+F 4 "Samtec" H 950 1950 50  0001 C CNN "Manufacturer"
+F 5 "SMA-J-P-H-ST-EM1" H 950 1950 50  0001 C CNN "Part Number"
+F 6 "SMA_END_LAUNCH" H 950 1950 50  0001 C CNN "Package"
+F 7 "SMA Connector Jack, Female Socket 50 Ohm Board Edge, End Launch Solder" H 950 1950 50  0001 C CNN "Description"
 	1    950  1950
 	1    0    0    -1
@@
 F 2 "samtec:SMA-J-P-H-ST-EM1" H 2650 1750 50  0001 L BNN
 F 3 "Connector SMA F 50Ohm Solder ST Edge Mount Gold Over Nickel Tray" H 2650 1750 50  0001 L BNN
-F 4 "None" H 2650 1750 50  0001 L BNN "Field4"
-F 5 "SMA-J-P-H-ST-EM1" H 2650 1750 50  0001 L BNN "Field5"
-F 6 "Good" H 2650 1750 50  0001 L BNN "Field6"
-F 7 "2.95 USD" H 2650 1750 50  0001 L BNN "Field7"
-F 8 "Samtec" H 2650 1750 50  0001 L BNN "Field8"
+F 4 "Samtec" H 2650 1750 50  0001 C CNN "Manufacturer"
+F 5 "SMA-J-P-H-ST-EM1" H 2650 1750 50  0001 C CNN "Part Number"
+F 6 "SMA_END_LAUNCH" H 2650 1750 50  0001 C CNN "Package"
+F 7 "SMA Connector Jack, Female Socket 50 Ohm Board Edge, End Launch Solder" H 2650 1750 50  0001 C CNN "Description"
 	1    2650 1750
 	1    0    0    -1
@@
 F 2 "samtec:SMA-J-P-H-ST-EM1" H 10200 2600 50  0001 L BNN
 F 3 "Connector SMA F 50Ohm Solder ST Edge Mount Gold Over Nickel Tray" H 10200 2600 50  0001 L BNN
-F 4 "None" H 10200 2600 50  0001 L BNN "Field4"
-F 5 "SMA-J-P-H-ST-EM1" H 10200 2600 50  0001 L BNN "Field5"
-F 6 "Good" H 10200 2600 50  0001 L BNN "Field6"
-F 7 "2.95 USD" H 10200 2600 50  0001 L BNN "Field7"
-F 8 "Samtec" H 10200 2600 50  0001 L BNN "Field8"
+F 4 "Samtec" H 10200 2600 50  0001 C CNN "Manufacturer"
+F 5 "SMA-J-P-H-ST-EM1" H 10200 2600 50  0001 C CNN "Part Number"
+F 6 "SMA_END_LAUNCH" H 10200 2600 50  0001 C CNN "Package"
+F 7 "SMA Connector Jack, Female Socket 50 Ohm Board Edge, End Launch Solder" H 10200 2600 50  0001 C CNN "Description"
 	1    10200 2600
 	-1   0    0    -1
@@
 F 2 "samtec:SMA-J-P-H-ST-EM1" H 6450 6750 50  0001 L BNN
 F 3 "Connector SMA F 50Ohm Solder ST Edge Mount Gold Over Nickel Tray" H 6450 6750 50  0001 L BNN
-F 4 "None" H 6450 6750 50  0001 L BNN "Field4"
-F 5 "SMA-J-P-H-ST-EM1" H 6450 6750 50  0001 L BNN "Field5"
-F 6 "Good" H 6450 6750 50  0001 L BNN "Field6"
-F 7 "2.95 USD" H 6450 6750 50  0001 L BNN "Field7"
-F 8 "Samtec" H 6450 6750 50  0001 L BNN "Field8"
+F 4 "Samtec" H 6450 6750 50  0001 C CNN "Manufacturer"
+F 5 "SMA-J-P-H-ST-EM1" H 6450 6750 50  0001 C CNN "Part Number"
+F 6 "SMA_END_LAUNCH" H 6450 6750 50  0001 C CNN "Package"
+F 7 "SMA Connector Jack, Female Socket 50 Ohm Board Edge, End Launch Solder" H 6450 6750 50  0001 C CNN "Description"
 	1    6450 6750
 	-1   0    0    -1
@@
 F 4 "Guerilla RF" H 2700 6850 50  0001 C CNN "Manufacturer"
 F 5 "GRF4142" H 2700 6850 50  0001 C CNN "Part Number"
+F 6 "RF Amplifier .1-3.8GHz GaAs Gain 16dB" H 2700 6850 50  0001 C CNN "Description"
 	1    2700 6850
 	1    0    0    -1
@@
 F 4 "Guerilla RF" H 5350 1850 50  0001 C CNN "Manufacturer"
 F 5 "GRF4142" H 5350 1850 50  0001 C CNN "Part Number"
+F 6 "RF Amplifier .1-3.8GHz GaAs Gain 16dB" H 5350 1850 50  0001 C CNN "Description"
 	1    5350 1850
 	1    0    0    -1

Commit message: Board is out for quote to several places.
Parts:
- M1, M2: value 2118706-2 -> DNP
Changed lines of the file:
@@
 P 8150 1200
 F 0 "M2" H 8225 1775 50  0000 C CNN
-F 1 "2118706-2" H 8225 1684 50  0000 C CNN
+F 1 "DNP" H 8225 1684 50  0000 C CNN
 F 2 "project_footprints:2118706-2" H 8150 1200 50  0001 C CNN
 F 3 "http://www.te.com/commerce/DocumentDelivery/DDEController?Action=showdoc&DocId=Customer+Drawing%7F2118706%7FA2%7Fpdf%7FEnglish%7FENG_CD_2118706_A2.pdf%7F2118706-2" H 8150 1200 50  0001 C CNN
 F 4 "TE Connectivity" H 8150 1200 50  0001 C CNN "Manufacturer"
-F 5 "2118706-2" H 8150 1200 50  0001 C CNN "Part Number"
+F 5 "2118706-2" H 8200 1150 50  0000 C CNN "Part Number"
 F 6 "RF Sheild" H 8150 1200 50  0001 C CNN "Description"
 	1    8150 1200
@@
 P 1300 5750
 F 0 "M1" H 1375 6325 50  0000 C CNN
-F 1 "2118706-2" H 1375 6234 50  0000 C CNN
+F 1 "DNP" H 1375 6234 50  0000 C CNN
 F 2 "project_footprints:2118706-2" H 1300 5750 50  0001 C CNN
 F 3 "http://www.te.com/commerce/DocumentDelivery/DDEController?Action=showdoc&DocId=Customer+Drawing%7F2118706%7FA2%7Fpdf%7FEnglish%7FENG_CD_2118706_A2.pdf%7F2118706-2" H 1300 5750 50  0001 C CNN
 F 4 "TE Connectivity" H 1300 5750 50  0001 C CNN "Manufacturer"
-F 5 "2118706-2" H 1300 5750 50  0001 C CNN "Part Number"
+F 5 "2118706-2" H 1400 5700 50  0000 C CNN "Part Number"
 F 6 "RF Sheild" H 1300 5750 50  0001 C CNN "Description"
 	1    1300 5750
