File: rf-section.sch (KiCad schematic (older format))
At the start: 54 parts, among them J4 SMA-J-P-H-ST-EM1, J5 SMA-J-P-H-ST-EM1, J7 SMA-J-P-H-ST-EM1, J8 SMA-J-P-H-ST-EM1, M1 DNP, M2 DNP, U12 SKY13414-485LF, U6 SKY13414-485LF, U7 GRF4142, U8 GRF4142

Commit message: The project footprints have been locally archived now. Now, all of the footprints are loacl within the project.
Parts:
- C12, C15, C16, C17, C18, C19, C20, C22, C23, C24, C25, C26, C27, C28, C29, C30, C31, C32, C33, C34, C35, C36, C37: footprint project_footprints:C_0402 -> project_footprints.pretty:C_0402
- D6, D7, D8, D9: footprint project_footprints:ONSEMI_0201_DSN2_153AF -> project_footprints.pretty:ONSEMI_0201_DSN2_153AF
- FL1, FL2, FL3: footprint project_footprints:SAW_3X3mm -> project_footprints.pretty:SAW_3X3mm
- J4, J5, J7, J8: footprint samtec:SMA-J-P-H-ST-EM1 -> project_footprints.pretty:SMA-J-P-H-ST-EM1
- L1, L2, L3, L4: footprint murata:L_0402 -> project_footprints.pretty:L_0402
- L5: footprint murata:INDC2520X100 -> project_footprints.pretty:INDC2520X100
- L6: footprint murata:FB_0402_NoSilk -> project_footprints.pretty:FB_0402_NoSilk
- M1, M2: footprint project_footprints:2118706-2 -> project_footprints.pretty:2118706-2
- R12, R14, R15, R16, R17, R21, R22, R25: footprint project_footprints:R_0402 -> project_footprints.pretty:R_0402
- U12, U6: footprint project_footprints:QFN45P200X200X55-15N -> project_footprints.pretty:QFN45P200X200X55-15N
- U7, U8: footprint guerilla_rf:DFN1.5MMX1.5MMX0.45MM-6 -> project_footprints.pretty:DFN1.5MMX1.5MMX0.45MM-6

Commit message: More dicking around with CMs
Parts:
- M1, M2: value DNP -> DNF
Changed lines of the file:
@@
 P 8150 1200
 F 0 "M2" H 8225 1775 50  0000 C CNN
-F 1 "DNP" H 8225 1684 50  0000 C CNN
+F 1 "DNF" H 8225 1684 50  0000 C CNN
 F 2 "project_footprints.pretty:2118706-2" H 8150 1200 50  0001 C CNN
 F 3 "http://www.te.com/commerce/DocumentDelivery/DDEController?Action=showdoc&DocId=Customer+Drawing%7F2118706%7FA2%7Fpdf%7FEnglish%7FENG_CD_2118706_A2.pdf%7F2118706-2" H 8150 1200 50  0001 C CNN
@@
 P 1300 5750
 F 0 "M1" H 1375 6325 50  0000 C CNN
-F 1 "DNP" H 1375 6234 50  0000 C CNN
+F 1 "DNF" H 1375 6234 50  0000 C CNN
 F 2 "project_footprints.pretty:2118706-2" H 1300 5750 50  0001 C CNN
 F 3 "http://www.te.com/commerce/DocumentDelivery/DDEController?Action=showdoc&DocId=Customer+Drawing%7F2118706%7FA2%7Fpdf%7FEnglish%7FENG_CD_2118706_A2.pdf%7F2118706-2" H 1300 5750 50  0001 C CNN
