File: pi-hat-lna.kicad_pcb (KiCad board)
At the start: 4 copper layers, 65 x 56 mm, 105 parts, among them J1 USB_B_Mini, J2 Conn_02x03_Odd_Even, J3 40HAT, J4 619540-1, J5 619540-1, J6 CONN_02X02, J7 619540-1, J8 619540-1, J9 CONN_01X02, Q1 DMG2305UX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

Commit message: Trimmed unnecessary parts from the Pi power circuitry. Now the Pi 5V is diode or'd with VBUS from the USB
Parts:
- removed C24: 100nF, project_footprints:C_0402
- removed C25, C27, C30, C31, C33, C36: 100pF, project_footprints:C_0402
- removed J6: CONN_02X02, project_footprints:PinHeader_2x02_P2.54mm_Vertical
- removed Q1: DMG2305UX, project_footprints:SOT-23
- removed Q2: DMMT5401, project_footprints:SOT-23-6
- removed R19, R20, R26, R27: 100, project_footprints:R_0402
- removed R23, R24: 22, project_footprints:R_0603_1608Metric_Pad0.84x1.00mm_HandSolder
- removed R7, R9: DNP, project_footprints:R_0603_1608Metric_Pad0.84x1.00mm_HandSolder
- removed U10, U13, U9: SKY13351-378LF, project_footprints:SKY_QFN6_1x1mm
- removed U11: SPF5122Z, project_footprints:DFN-8
- added C12: 100pF, project_footprints:C_0402, F.Cu at (96.6, 88.2)
- added D10: BAT165, project_footprints:D_SOD-323, F.Cu at (69.6, 64.2)
- added D11: BAT165, project_footprints:D_SOD-323, F.Cu at (71.4, 70.9)
- added L3: 12nH, project_footprints:LQW15A, F.Cu at (129.2, 96.4)
- added L4: 12nH, project_footprints:LQW15A, F.Cu at (124.9, 92.3)
- added M1: 2118706-2, project_footprints:2118706-2, F.Cu at (127.0, 93.0)
- added M2: 2118706-2, project_footprints:2118706-2, F.Cu at (52.0, 93.0)
- C15: value 100pF -> 100nF
- FL3: value TA1090EC -> SF2275E; footprint project_footprints:SAW_3.8X3.8MM -> project_footprints:SAW_3X3mm
- L1, L2: value 150nH -> 12nH; footprint project_footprints:L_0603 -> project_footprints:LQW15A
- R13, R18: value 100 -> 374
- U7: value SKY13351-378LF -> GRF4042; footprint project_footprints:SKY_QFN6_1x1mm -> project_footprints:QFN-12_EP_2x2_Pitch0.5mm
- U8: value SPF5122Z -> GRF4042; footprint project_footprints:DFN-8 -> project_footprints:QFN-12_EP_2x2_Pitch0.5mm
- moved C19 42.8 mm to (131.2, 103.7), turned to 180 degrees
- moved C23 41.3 mm to (91.4, 102.9), turned to 180 degrees
- moved U8 37.2 mm to (127.9, 93.3), turned to 90 degrees
- moved L2 36.5 mm to (96.3, 97.4)
- moved C21 32.5 mm to (124.7, 88.1), turned to 180 degrees
- moved C35 14.5 mm to (114.7, 82.8)
- moved C15 13.6 mm to (98.0, 98.0), turned to 90 degrees
- moved C18 12.1 mm to (107.2, 83.1)
- moved U6 11.3 mm to (104.0, 82.0), turned to 90 degrees
- moved U12 11.2 mm to (118.0, 84.0), turned to 270 degrees
- moved R13 11.0 mm to (96.3, 95.9), turned to 180 degrees
- moved C32 10.6 mm to (123.0, 92.9)
- moved R18 10.6 mm to (125.0, 93.8), turned to 0 degrees
- moved U7 9.28 mm to (93.0, 96.9), turned to 270 degrees
- moved R14 8.25 mm to (105.0, 99.5), turned to 270 degrees
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Connections:
- C15 pad 1: Net-(C15-Pad1) -> GND
- C15 pad 2: Net-(C15-Pad2) -> +3.3VA
- C2 pad 1: VBUS -> Net-(C2-Pad1)
- D7 pad 2: Net-(C23-Pad2) -> Net-(C19-Pad1)
- D8 pad 2: Net-(C30-Pad1) -> Net-(C23-Pad2)
- J5 pad 1: Net-(C23-Pad2) -> Net-(C19-Pad1)
- J7 pad 1: Net-(C30-Pad1) -> Net-(C23-Pad2)
- L1 pad 1: +3.3VA -> Net-(C12-Pad2)
- L1 pad 2: Net-(C25-Pad2) -> GND
- L2 pad 2: Net-(C33-Pad2) -> Net-(L2-Pad2)
- R12 pad 1: Net-(R12-Pad1) -> /avr-usb/BYP_LNA2
- R12 pad 2: /avr-usb/BYP_LNA2 -> Net-(R12-Pad2)
- R13 pad 1: /avr-usb/BYP_LNA2_N -> +3.3VA
- R17 pad 1: Net-(R17-Pad1) -> /avr-usb/BYP_LNA1
- R17 pad 2: /avr-usb/BYP_LNA1 -> Net-(R17-Pad2)
- R18 pad 1: /avr-usb/BYP_LNA1_N -> +3.3VA
- R29 pad 1: /P3V3 -> +3V3
- R6 pad 1: /P3V3 -> +3V3
- R8 pad 1: /P3V3 -> +3V3
- U12 pad 13: Net-(C36-Pad1) -> Net-(C21-Pad2)
- U2 pad 8: /P3V3 -> +3V3
- U3 pad 1: VBUS -> Net-(C2-Pad1)
- U3 pad 3: VBUS -> Net-(C2-Pad1)
- U5 pad 13: /avr-usb/BYP_LNA1_N -> (no net)
- U5 pad 28: /avr-usb/BYP_LNA2_N -> (no net)
- U6 pad 13: Net-(C15-Pad2) -> Net-(C12-Pad1)
- U7 pad 1: Net-(C19-Pad2) -> Net-(R12-Pad2)
- U7 pad 3: Net-(C21-Pad2) -> Net-(C12-Pad2)
- U7 pad 4: Net-(R12-Pad1) -> GND
- U7 pad 5: Net-(C15-Pad1) -> GND
- U7 pad 6: Net-(R13-Pad2) -> GND
- U8 pad 1: GND -> Net-(R17-Pad2)
- U8 pad 2: Net-(C19-Pad1) -> GND
- U8 pad 3: Net-(C19-Pad1) -> Net-(C19-Pad2)
- U8 pad 6: Net-(C25-Pad2) -> GND
- U8 pad 7: Net-(C25-Pad2) -> Net-(C21-Pad1)
Routing:
- net /P3V3: track 31.3 -> 0.00 mm
- net /P5V: track 8.71 -> 0.00 mm
- net +3V3: track 0.00 -> 8.18 mm
- net Net-(Q1-Pad1): track 6.02 -> 0.00 mm
- net /P5V_HAT: track 3.77 -> 0.00 mm
- net Net-(Q2-Pad1): track 3.37 -> 0.00 mm
- net /P3V3_HAT: track 2.88 -> 0.00 mm

Commit message: Can now power via: 1. USB 2. R-Pi 3. Bias TEE
Parts:
- added C24: 1uF, project_footprints:C_0402, F.Cu at (89.4, 108.4)
- added D12: BAT165, project_footprints:D_SOD-323, F.Cu at (90.5, 70.6)
- added J6: TAG-Connect, Connectors:Tag-Connect_TC2030-IDC-NL, F.Cu at (122.0, 101.8)
- added L5: 1uH, murata:INDC2520X100, F.Cu at (90.4, 104.7)
- added SW1: TL3305AF160QG, e_switch:TL3305AF160QG, F.Cu at (129.2, 111.7)
- J2: value Conn_02x03_Odd_Even -> .1" Header
- moved C4 45.4 mm to (94.0, 72.9)
- moved C2 45.3 mm to (96.0, 69.6), turned to 0 degrees
- moved U3 43.9 mm to (96.4, 72.1), turned to 270 degrees
- moved M2 43.0 mm to (95.0, 92.0), turned to 90 degrees
- moved C6 39.1 mm to (97.0, 74.6)
- moved C1 35.1 mm to (101.6, 69.9), turned to 0 degrees
- moved C3 33.1 mm to (99.9, 73.2), turned to 90 degrees
- moved U1 31.7 mm to (102.3, 72.4), turned to 270 degrees
- moved C5 26.9 mm to (102.7, 75.0)
- moved D10 21.5 mm to (90.6, 68.5), turned to 180 degrees
- moved D11 19.2 mm to (90.5, 72.6), turned to 180 degrees
- moved R4 17.5 mm to (120.0, 97.6), turned to 180 degrees
- moved D4 13.7 mm to (120.0, 99.0), turned to 0 degrees
- moved R10 12.7 mm to (123.3, 104.5), turned to 180 degrees
- moved D5 10.7 mm to (113.2, 109.3), turned to 90 degrees
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Connections:
- C1 pad 1: VBUS -> +5V
- C2 pad 1: Net-(C2-Pad1) -> +5V
- D10 pad 1: Net-(C2-Pad1) -> +5V
- D11 pad 1: Net-(C2-Pad1) -> +5V
- J2 pad 1: /avr-usb/MISO -> /avr-usb/PC0
- J2 pad 2: /avr-usb/VCC -> /avr-usb/PC2
- J2 pad 3: /avr-usb/SCK -> /avr-usb/PC1
- J2 pad 4: /avr-usb/MOSI -> /avr-usb/PC3
- J2 pad 5: /avr-usb/~RESET -> /avr-usb/PC4
- J3 pad 1: /P3V3_HAT -> (no net)
- R5 pad 1: /avr-usb/LED_GRN -> Net-(D5-Pad2)
- R5 pad 2: Net-(D5-Pad2) -> /avr-usb/LED_GRN
- U1 pad 1: VBUS -> +5V
- U1 pad 3: VBUS -> +5V
- U3 pad 1: Net-(C2-Pad1) -> +5V
- U3 pad 3: Net-(C2-Pad1) -> +5V
- U5 pad 1: /avr-usb/SWA_V2 -> /avr-usb/LED_GRN
- U5 pad 10: /avr-usb/SWB_V2 -> /avr-usb/PC1
- U5 pad 11: /avr-usb/SWB_V3 -> /avr-usb/PC2
- U5 pad 12: /avr-usb/LED_GRN -> (no net)
- U5 pad 13: (no net) -> /avr-usb/BTN
- U5 pad 2: /avr-usb/SWA_V3 -> (no net)
- U5 pad 23: (no net) -> /avr-usb/SWB_V1
- U5 pad 24: (no net) -> /avr-usb/SWB_V2
- U5 pad 25: (no net) -> /avr-usb/SWB_V3
- U5 pad 26: (no net) -> /avr-usb/SWA_V1
- U5 pad 27: /avr-usb/BYP_LNA2 -> /avr-usb/SWA_V2
- U5 pad 28: (no net) -> /avr-usb/BYP_LNA2
- U5 pad 32: /avr-usb/SWA_V1 -> /avr-usb/SWA_V3
- U5 pad 7: (no net) -> /avr-usb/PC3
- U5 pad 8: (no net) -> /avr-usb/PC4
- U5 pad 9: /avr-usb/SWB_V1 -> /avr-usb/PC0
Routing:
- removed copper zone on B.Cu, net /P3V3_HAT
- removed copper zone on F.Cu, net /P5V
- removed copper zone on B.Cu, net /P5V_HAT
- removed copper zone on F.Cu, net /P5V_HAT
- removed copper zone on F.Cu, net GND

Commit message: Finally have the stackup
Parts:
- removed J2: .1" Header, project_footprints:FRAMATOME_67997-206HLF
- added D13: SML-LX0402SUGC-TR, project_footprints:LED_0402, F.Cu at (116.3, 114.0)
- added D14: SML-LX0402SUGC-TR, project_footprints:LED_0402, F.Cu at (123.8, 114.0)
- added D15: SML-LX0402SUGC-TR, project_footprints:LED_0402, F.Cu at (118.8, 114.0)
- added D16: SML-LX0402SUGC-TR, project_footprints:LED_0402, F.Cu at (121.3, 114.0)
- added R19: 1K, project_footprints:R_0402, F.Cu at (116.3, 111.0)
- added R20: 1K, project_footprints:R_0402, F.Cu at (123.8, 111.0)
- added R23: 1K, project_footprints:R_0402, F.Cu at (118.8, 111.0)
- added R24: 1K, project_footprints:R_0402, F.Cu at (121.3, 111.0)
- added R7: 3.9K, project_footprints:R_0402, F.Cu at (113.6, 99.2)
- added R9: 3.9K, project_footprints:R_0402, F.Cu at (112.4, 99.2)
- J4, J5, J7, J8: value 619540-1 -> VAL**; footprint project_footprints:619540-1 -> samtec:SMA-J-P-H-ST-EM1
- R11, R29, R6, R8: footprint project_footprints:R_0603_1608Metric_Pad0.84x1.00mm_HandSolder -> project_footprints:R_0402
- SW1: value TL3305AF160QG -> VAL**
- U7, U8: value GRF4042 -> GRF4142
- moved J9 12.7 mm to (126.0, 71.0)
- moved R11 8.92 mm to (127.1, 68.5)
- moved R25 6.35 mm to (119.1, 95.9)
- moved R21 6.28 mm to (117.8, 95.9)
- moved R22 6.28 mm to (116.6, 95.9)
- moved D5 4.76 mm to (113.8, 114.0)
- moved R5 3.72 mm to (113.8, 111.0)
- moved J5 2.64 mm to (141.6, 104.0), turned to 90 degrees
- moved J8 2.64 mm to (141.6, 77.0), turned to 90 degrees
- moved J4 2.56 mm to (80.4, 77.0), turned to 270 degrees
- moved J7 2.56 mm to (80.4, 104.0), turned to 270 degrees
- moved R15 2.04 mm to (108.5, 99.8)
- moved R16 2.04 mm to (109.7, 99.8)
- moved R14 1.95 mm to (110.9, 99.8)
- moved SW1 1.49 mm to (130.0, 113.0), turned to 0 degrees
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Connections:
- net /avr-usb/LED_GRN renamed /avr-usb/LED1
- J3 pad 3: (no net) -> /PI_SDA
- J3 pad 5: (no net) -> /PI_SCL
- R11 pad 1: Net-(J9-Pad2) -> GND
- R11 pad 2: GND -> Net-(J9-Pad2)
- U5 pad 10: /avr-usb/PC1 -> /avr-usb/BTN
- U5 pad 11: /avr-usb/PC2 -> /avr-usb/BYP_LNA1
- U5 pad 12: (no net) -> /avr-usb/SWB_V1
- U5 pad 13: /avr-usb/BTN -> /avr-usb/SWB_V2
- U5 pad 14: /avr-usb/BYP_LNA1 -> /avr-usb/SWB_V3
- U5 pad 2: (no net) -> /avr-usb/LED2
- U5 pad 23: /avr-usb/SWB_V1 -> /PI_SDA
- U5 pad 24: /avr-usb/SWB_V2 -> /PI_SCL
- U5 pad 25: /avr-usb/SWB_V3 -> /avr-usb/SWA_V1
- U5 pad 26: /avr-usb/SWA_V1 -> /avr-usb/SWA_V2
- U5 pad 27: /avr-usb/SWA_V2 -> /avr-usb/SWA_V3
- U5 pad 32: /avr-usb/SWA_V3 -> (no net)
- U5 pad 7: /avr-usb/PC3 -> /avr-usb/LED4
- U5 pad 8: /avr-usb/PC4 -> /avr-usb/LED5
- U5 pad 9: /avr-usb/PC0 -> /avr-usb/LED3
Routing:
- net Net-(J9-Pad2): track 9.58 -> 18.0 mm
- net GND: track 0.00 -> 2.97 mm
- net +3V3: track 8.18 -> 6.99 mm
Other:
- board text added: "0.062"
- board text added: "1 oz Cu"
- board text removed: "If you want to use an SMT 40-pin header, please move the top edge up by 0.5mm and locate the header in the same location as the current TH part."

Commit message: I think the layout is ready for review
Parts:
- removed C21: 100pF, project_footprints:C_0402
- removed R13, R18: 374, project_footprints:R_0402
- added C25: 30pF, project_footprints:C_0402, F.Cu at (92.0, 89.3)
- added C27: DNF, project_footprints:C_0402, F.Cu at (91.5, 91.1)
- added C30: 1pF, project_footprints:C_0402, F.Cu at (91.4, 96.9)
- added C31: 30pF, project_footprints:C_0402, F.Cu at (133.0, 94.6)
- added C33: DNF, project_footprints:C_0402, F.Cu at (133.6, 92.8)
- added C36: 1pF, project_footprints:C_0402, F.Cu at (133.6, 87.5)
- added C37: 100pF, project_footprints:C_0402, F.Cu at (133.1, 84.5)
- added L6: BLM15AG121SN1D, murata:FB_0402_NoSilk, F.Cu at (86.0, 104.3)
- J6: value TAG-Connect -> 2x3 0.1" HEADER; footprint Connectors:Tag-Connect_TC2030-IDC-NL -> amphenol:FRAMATOME_67997-206HLF
- L1, L3: value 12nH -> 22nH; footprint project_footprints:LQW15A -> murata:L_0402
- L2, L4: value 12nH -> 39nH; footprint project_footprints:LQW15A -> murata:L_0402
- R12, R17: value 100 -> 1.4K
- U7, U8: footprint project_footprints:QFN-12_EP_2x2_Pitch0.5mm -> guerilla_rf:DFN1.5MMX1.5MMX0.45MM-6
- moved D16 40.5 mm to (109.1, 75.3), turned to 0 degrees
- moved D12 37.3 mm to (92.0, 107.8)
- moved R24 37.0 mm to (111.3, 75.3), turned to 0 degrees
- moved D5 36.4 mm to (83.5, 93.7)
- moved D11 34.3 mm to (96.6, 106.3), turned to 270 degrees
- moved R5 33.6 mm to (85.0, 93.6), turned to 270 degrees
- moved C4 32.9 mm to (108.2, 102.5), turned to 0 degrees
- moved C2 31.9 mm to (103.9, 100.5), turned to 90 degrees
- moved D15 31.6 mm to (110.5, 83.5)
- moved R23 30.1 mm to (111.4, 81.8), turned to 0 degrees
- moved U3 29.7 mm to (106.4, 100.0), turned to 0 degrees
- moved C6 27.7 mm to (108.9, 99.6), turned to 270 degrees
- moved D14 25.7 mm to (140.3, 94.3)
- moved R20 22.7 mm to (139.0, 94.1), turned to 270 degrees
- moved D13 20.2 mm to (108.1, 95.6), turned to 0 degrees
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Connections:
- J3 pad 1: (no net) -> /P3V3_HAT
- L2 pad 2: Net-(L2-Pad2) -> Net-(C23-Pad1)
- L4 pad 2: Net-(L4-Pad2) -> Net-(C36-Pad1)
- L5 pad 2: Net-(C23-Pad2) -> Net-(L5-Pad2)
- R12 pad 1: /avr-usb/BYP_LNA2 -> Net-(R12-Pad1)
- R12 pad 2: Net-(R12-Pad2) -> /avr-usb/BYP_LNA2
- R17 pad 1: /avr-usb/BYP_LNA1 -> Net-(R17-Pad1)
- R17 pad 2: Net-(R17-Pad2) -> /avr-usb/BYP_LNA1
- R29 pad 1: +3V3 -> /P3V3_HAT
- R6 pad 1: +3V3 -> /P3V3_HAT
- R8 pad 1: +3V3 -> /P3V3_HAT
- U2 pad 8: +3V3 -> /P3V3_HAT
- U5 pad 10: /avr-usb/BTN -> /avr-usb/LED3
- U5 pad 12: /avr-usb/SWB_V1 -> /avr-usb/SWB_V3
- U5 pad 14: /avr-usb/SWB_V3 -> /avr-usb/SWB_V1
- U5 pad 25: /avr-usb/SWA_V1 -> /avr-usb/SWA_V3
- U5 pad 27: /avr-usb/SWA_V3 -> /avr-usb/SWA_V1
- U5 pad 9: /avr-usb/LED3 -> /avr-usb/BTN
- U7 pad 1: Net-(R12-Pad2) -> Net-(R12-Pad1)
- U7 pad 3: Net-(C12-Pad2) -> Net-(C25-Pad2)
- U7 pad 4: GND -> Net-(C23-Pad1)
- U8 pad 1: Net-(R17-Pad2) -> Net-(R17-Pad1)
- U8 pad 3: Net-(C19-Pad2) -> Net-(C31-Pad2)
- U8 pad 4: GND -> Net-(C36-Pad1)
Routing:
- net +5V: track 0.00 -> 56.1 mm, vias 0 -> 19
- net /PI_SDA: track 0.00 -> 52.3 mm, vias 0 -> 1
- net /PI_SCL: track 0.00 -> 47.5 mm, vias 0 -> 1
- net +3V3: track 6.99 -> 47.7 mm, vias 0 -> 6
- net /P3V3_HAT: track 0.00 -> 38.4 mm
- net /avr-usb/LED5: track 0.00 -> 35.2 mm, vias 0 -> 2
- net /avr-usb/LED1: track 0.00 -> 34.2 mm, vias 0 -> 2
- net GND: track 2.97 -> 33.8 mm, vias 0 -> 299
- net /avr-usb/LED4: track 0.00 -> 28.8 mm, vias 0 -> 2
- net /avr-usb/LED3: track 0.00 -> 28.6 mm, vias 0 -> 2
- net +3.3VA: track 0.00 -> 27.7 mm, vias 0 -> 13
- net /avr-usb/SWA_V1: track 0.00 -> 26.6 mm, vias 0 -> 2
- net VBUS: track 0.00 -> 25.9 mm, vias 0 -> 1
- net /avr-usb/SWB_V3: track 0.00 -> 25.1 mm, vias 0 -> 2
- net /avr-usb/SWA_V2: track 0.00 -> 23.9 mm, vias 0 -> 2
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- added copper zone on In2.Cu, net +3.3VA
- added copper zone on In2.Cu, net +5V
- added copper zone on In2.Cu, net /P5V_HAT
- added copper zone on F.Cu, net GND
- added copper zone on In1.Cu, net GND
- removed copper zone on In2.Cu, net GND
Other:
- net class Default: clearance 0.2 -> 0.1524
- rule trace_clearance: 0.2 -> 0.1524
- board text added: "50 Ohm trace = 18.5 mil (0.47 mm)"
- board text added: "9.3 mil ?"
- board text added: "LNA1"
- board text added: "LNA1 OUT"
- board text added: "LNA2"
- board text added: "LNA2 IN"
- board text added: "RF IN"
- board text added: "RF OUT"
- board text removed: "This is a HAT compatible PCB starting design based on the official Raspberry Pi specs at: https://github.com/raspberrypi/hats/blob/master/designguide.md Currently the camera slot and display cutout are not here. See the schematic for the details on the EEPROM and power setup. This board does have the correct components for powering the Pi via the HAT. If you need the Pi to provide 5V or 3.3V, ple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"
