File: pi-hat-lna.kicad_pcb (KiCad board)
At the start: 4 copper layers, 65 x 56 mm, 109 parts, among them J1 USB_B_Mini, J3 DNF, J4 SMA-J-P-H-ST-EM1, J5 SMA-J-P-H-ST-EM1, J6 2x3 0.1" HEADER, J7 SMA-J-P-H-ST-EM1, J8 SMA-J-P-H-ST-EM1, J9 CONN_01X02, M1 2118706-2, M2 2118706-2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

Commit message: The project footprints have been locally archived now. Now, all of the footprints are loacl within the project.
Parts:
- J4, J5, J7, J8: value SMA-J-P-H-ST-EM1 -> VAL**
- SW1: value TL3305AF160QG -> VAL**
Changed lines of the file:
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@@
       (effects (font (size 0.8 0.8) (thickness 0.15)))
     )
-    (fp_text value TL3305AF160QG (at 0.175614 4.88242) (layer F.SilkS) hide
+    (fp_text value VAL** (at 0.175614 4.88242) (layer F.SilkS) hide
       (effects (font (size 0.5 0.5) (thickness 0.09)))
     )
@@
       (effects (font (size 0.8 0.8) (thickness 0.15)))
     )
-    (fp_text value SMA-J-P-H-ST-EM1 (at -0.225387 12.3855 270) (layer F.SilkS) hide
+    (fp_text value VAL** (at -0.225387 12.3855 270) (layer F.SilkS) hide
       (effects (font (size 1.00166 1.00166) (thickness 0.05)))
     )
@@
       (effects (font (size 0.8 0.8) (thickness 0.15)))
     )
-    (fp_text value SMA-J-P-H-ST-EM1 (at -0.225387 12.3855 90) (layer F.SilkS) hide
+    (fp_text value VAL** (at -0.225387 12.3855 90) (layer F.SilkS) hide
       (effects (font (size 1.00166 1.00166) (thickness 0.05)))
     )
@@
       (effects (font (size 0.8 0.8) (thickness 0.15)))
     )
-    (fp_text value SMA-J-P-H-ST-EM1 (at -0.225387 12.3855 270) (layer F.SilkS) hide
+    (fp_text value VAL** (at -0.225387 12.3855 270) (layer F.SilkS) hide
       (effects (font (size 1.00166 1.00166) (thickness 0.05)))
     )
@@
       (effects (font (size 0.8 0.8) (thickness 0.15)))
     )
-    (fp_text value SMA-J-P-H-ST-EM1 (at 5.78 -4.5 90) (layer F.SilkS) hide
+    (fp_text value VAL** (at 5.78 -4.5 90) (layer F.SilkS) hide
       (effects (font (size 1.00166 1.00166) (thickness 0.05)))
     )
