File: pi-hat-lna.sch (KiCad schematic (older format))
At the start: 18 parts, among them J3 40HAT, J6 CONN_02X02, J9 CONN_01X02, Q1 DMG2305UX, Q2 DMMT5401, U2 CAT24C32

Commit message: Almost all 3D models have been added. Rough parts placement complete.
Parts:
- J3: footprint Connector_PinSocket_2.54mm:PinSocket_2x20_P2.54mm_Vertical -> project_footprints:PinSocket_2x20_P2.54mm_Vertical
- J6: footprint Connector_PinHeader_2.54mm:PinHeader_2x02_P2.54mm_Vertical -> project_footprints:PinHeader_2x02_P2.54mm_Vertical
- J9: footprint Connector_PinHeader_2.54mm:PinHeader_1x02_P2.54mm_Vertical -> project_footprints:PinHeader_1x02_P2.54mm_Vertical
- Q1: footprint Package_TO_SOT_SMD:SOT-23 -> project_footprints:SOT-23
- Q2: footprint Package_TO_SOT_SMD:SOT-23-6 -> project_footprints:SOT-23-6
- R11, R23, R24, R29, R6, R7, R8, R9: footprint Resistor_SMD:R_0603_1608Metric_Pad0.84x1.00mm_HandSolder -> project_footprints:R_0603_1608Metric_Pad0.84x1.00mm_HandSolder
- U2: footprint Package_SOIC:SOIC-8_3.9x4.9mm_P1.27mm -> project_footprints:SOIC-8_3.9x4.9mm_P1.27mm
Changed lines of the file:
@@
 F 0 "J3" H 2950 2350 50  0000 C CNN
 F 1 "40HAT" H 2300 2350 50  0000 C CNN
-F 2 "Connector_PinSocket_2.54mm:PinSocket_2x20_P2.54mm_Vertical" H 2600 2450 50  0001 C CNN
+F 2 "project_footprints:PinSocket_2x20_P2.54mm_Vertical" H 2600 2450 50  0001 C CNN
 F 3 "" H 1900 2250 50  0000 C CNN
 	1    2600 2250
@@
 F 0 "J6" H 6050 4750 50  0000 C CNN
 F 1 "CONN_02X02" H 6050 4450 50  0000 C CNN
-F 2 "Connector_PinHeader_2.54mm:PinHeader_2x02_P2.54mm_Vertical" H 6050 3400 50  0001 C CNN
+F 2 "project_footprints:PinHeader_2x02_P2.54mm_Vertical" H 6050 3400 50  0001 C CNN
 F 3 "" H 6050 3400 50  0000 C CNN
 	1    6050 4600
@@
 F 0 "Q1" V 6300 2550 50  0000 R CNN
 F 1 "DMG2305UX" V 6300 2350 50  0000 R CNN
-F 2 "Package_TO_SOT_SMD:SOT-23" H 6350 2500 50  0001 C CNN
+F 2 "project_footprints:SOT-23" H 6350 2500 50  0001 C CNN
 F 3 "" H 6150 2400 50  0000 C CNN
 	1    6150 2400
@@
 F 0 "Q2" H 6050 3075 50  0000 L CNN
 F 1 "DMMT5401" H 6050 3000 50  0000 L CNN
-F 2 "Package_TO_SOT_SMD:SOT-23-6" H 6050 2925 50  0000 L CIN
+F 2 "project_footprints:SOT-23-6" H 6050 2925 50  0000 L CIN
 F 3 "" H 5850 3000 50  0000 L CNN
 	1    5850 3000
@@
 F 0 "Q2" H 6650 3075 50  0000 L CNN
 F 1 "DMMT5401" H 6650 3000 50  0000 L CNN
-F 2 "Package_TO_SOT_SMD:SOT-23-6" H 6650 2925 50  0000 L CIN
+F 2 "project_footprints:SOT-23-6" H 6650 2925 50  0000 L CIN
 F 3 "" H 6450 3000 50  0000 L CNN
 	2    6450 3000
@@
 F 0 "R23" V 5830 3600 50  0000 C CNN
 F 1 "22" V 5750 3600 50  0000 C CNN
-F 2 "Resistor_SMD:R_0603_1608Metric_Pad0.84x1.00mm_HandSolder" V 5680 3600 50  0001 C CNN
+F 2 "project_footprints:R_0603_1608Metric_Pad0.84x1.00mm_HandSolder" V 5680 3600 50  0001 C CNN
 F 3 "" H 5750 3600 50  0001 C CNN
 F 4 "Yageo" H -9800 -10750 50  0001 C CNN "MFR"
@@
 F 0 "R24" V 6630 3600 50  0000 C CNN
 F 1 "22" V 6550 3600 50  0000 C CNN
-F 2 "Resistor_SMD:R_0603_1608Metric_Pad0.84x1.00mm_HandSolder" V 6480 3600 50  0001 C CNN
+F 2 "project_footprints:R_0603_1608Metric_Pad0.84x1.00mm_HandSolder" V 6480 3600 50  0001 C CNN
 F 3 "" H 6550 3600 50  0001 C CNN
 F 4 "Yageo" H -9000 -10950 50  0001 C CNN "MFR"
@@
 F 0 "U2" H 2450 6200 50  0000 C CNN
 F 1 "CAT24C32" H 1850 6200 50  0000 C CNN
-F 2 "Package_SOIC:SOIC-8_3.9x4.9mm_P1.27mm" H 2100 5850 50  0001 C CNN
+F 2 "project_footprints:SOIC-8_3.9x4.9mm_P1.27mm" H 2100 5850 50  0001 C CNN
 F 3 "" H 2100 5850 50  0000 C CNN
 	1    2100 5850
@@
 F 0 "R6" V 2430 7400 50  0000 C CNN
 F 1 "3.9K" V 2350 7400 50  0000 C CNN
-F 2 "Resistor_SMD:R_0603_1608Metric_Pad0.84x1.00mm_HandSolder" V 2280 7400 50  0001 C CNN
+F 2 "project_footprints:R_0603_1608Metric_Pad0.84x1.00mm_HandSolder" V 2280 7400 50  0001 C CNN
 F 3 "" H 2350 7400 50  0001 C CNN
 F 4 "Yageo" H -13200 -6950 50  0001 C CNN "MFR"
@@
 F 0 "R8" V 2430 7650 50  0000 C CNN
 F 1 "3.9K" V 2350 7650 50  0000 C CNN
-F 2 "Resistor_SMD:R_0603_1608Metric_Pad0.84x1.00mm_HandSolder" V 2280 7650 50  0001 C CNN
+F 2 "project_footprints:R_0603_1608Metric_Pad0.84x1.00mm_HandSolder" V 2280 7650 50  0001 C CNN
 F 3 "" H 2350 7650 50  0001 C CNN
 F 4 "Yageo" H -13200 -6700 50  0001 C CNN "MFR"
@@
 F 0 "J9" H 750 6250 50  0000 C CNN
 F 1 "CONN_01X02" V 850 6100 50  0000 C CNN
-F 2 "Connector_PinHeader_2.54mm:PinHeader_1x02_P2.54mm_Vertical" H 750 6100 50  0001 C CNN
+F 2 "project_footprints:PinHeader_1x02_P2.54mm_Vertical" H 750 6100 50  0001 C CNN
 F 3 "" H 750 6100 50  0000 C CNN
 	1    750  6100
@@
 F 0 "R29" V 1630 6250 50  0000 C CNN
 F 1 "10K" V 1550 6250 50  0000 C CNN
-F 2 "Resistor_SMD:R_0603_1608Metric_Pad0.84x1.00mm_HandSolder" V 1480 6250 50  0001 C CNN
+F 2 "project_footprints:R_0603_1608Metric_Pad0.84x1.00mm_HandSolder" V 1480 6250 50  0001 C CNN
 F 3 "" H 1550 6250 50  0001 C CNN
 F 4 "Yageo" H -14000 -8100 50  0001 C CNN "MFR"
@@
 F 0 "R7" V 6180 4300 50  0000 C CNN
 F 1 "DNP" V 6100 4300 50  0000 C CNN
-F 2 "Resistor_SMD:R_0603_1608Metric_Pad0.84x1.00mm_HandSolder" V 6030 4300 50  0001 C CNN
+F 2 "project_footprints:R_0603_1608Metric_Pad0.84x1.00mm_HandSolder" V 6030 4300 50  0001 C CNN
 F 3 "" H 6100 4300 50  0001 C CNN
 F 4 "Yageo" H -9450 -10050 50  0001 C CNN "MFR"
@@
 F 0 "R9" V 6180 4950 50  0000 C CNN
 F 1 "DNP" V 6100 4950 50  0000 C CNN
-F 2 "Resistor_SMD:R_0603_1608Metric_Pad0.84x1.00mm_HandSolder" V 6030 4950 50  0001 C CNN
+F 2 "project_footprints:R_0603_1608Metric_Pad0.84x1.00mm_HandSolder" V 6030 4950 50  0001 C CNN
 F 3 "" H 6100 4950 50  0001 C CNN
 F 4 "Yageo" H -9450 -9400 50  0001 C CNN "MFR"
@@
 F 0 "R11" V 1380 6100 50  0000 C CNN
 F 1 "DNP" V 1300 6100 50  0000 C CNN
-F 2 "Resistor_SMD:R_0603_1608Metric_Pad0.84x1.00mm_HandSolder" V 1230 6100 50  0001 C CNN
+F 2 "project_footprints:R_0603_1608Metric_Pad0.84x1.00mm_HandSolder" V 1230 6100 50  0001 C CNN
 F 3 "" H 1300 6100 50  0001 C CNN
 F 4 "Yageo" H -14250 -8250 50  0001 C CNN "MFR"
@@
 NoConn ~ 2000 3750
 NoConn ~ 2000 3650
+$Comp
+L power:PWR_FLAG #FLG0101
+U 1 1 5B839C32
+P 2100 5350
+F 0 "#FLG0101" H 2100 5425 50  0001 C CNN
+F 1 "PWR_FLAG" V 2100 5478 50  0000 L CNN
+F 2 "" H 2100 5350 50  0001 C CNN
+F 3 "~" H 2100 5350 50  0001 C CNN
+	1    2100 5350
+	0    -1   -1   0
+$EndComp
+Connection ~ 2100 5350
 $EndSCHEMATC

Commit message: Trimmed unnecessary parts from the Pi power circuitry. Now the Pi 5V is diode or'd with VBUS from the USB
Parts:
- removed J6: CONN_02X02, project_footprints:PinHeader_2x02_P2.54mm_Vertical, symbol Connector_Generic:Conn_02x02_Odd_Even
- removed Q1: DMG2305UX, project_footprints:SOT-23, symbol raspberrypi_hat:DMG2305UX
- removed Q2: DMMT5401, project_footprints:SOT-23-6, symbol raspberrypi_hat:DMMT5401
- removed R23, R24: 22, project_footprints:R_0603_1608Metric_Pad0.84x1.00mm_HandSolder, symbol Device:R
- removed R7, R9: DNP, project_footprints:R_0603_1608Metric_Pad0.84x1.00mm_HandSolder, symbol Device:R
- added C1, C2, C5, C6: 1uF, project_footprints:C_0402, symbol Device:C
- added C3, C4: 100nF, project_footprints:C_0402, symbol Device:C
- added D10, D11: BAT165, project_footprints:D_SOD-323, symbol Diode:B160-E3
- added U1, U3: TPS73233DBVR, project_footprints:SOT-23-5, symbol Regulator_Linear:ADP7142AUZJ
Connections:
- net labels added: +3.3V, +3.3VA, VBUS
- net labels removed: P3V3, P5V
- wire segments 92 -> 87
Other:
- note added: "analog\nsupply"
- note added: "digital\nsupply"
- note removed: "5V Powered HAT Protection"
- note removed: "FLEXIBLE POWER SELECTION"
- note removed: "HAT spec indicates to NEVER\npower the 3.3V pins on the Raspberry Pi \nfrom the HAT header. Only connect the 3.3V\npower from the Pi if the HAT does not have\n3.3V on board.\n\nIF you are designing a board that could\neither be powered by the Pi or from the HAT\nthe jumpers here can be used.\n\nIn most cases, either design the HAT \nto provide the 5V to the Pi and use the\nprotection circuit abov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"
- note removed: "This is the recommended 5V rail protection for \na HAT with power going to the Pi.\nSee https://github.com/raspberrypi/hats/blob/master/designguide.md#back-powering-the-pi-via-the-j8-gpio-header"

Commit message: Can now power via: 1. USB 2. R-Pi 3. Bias TEE
Parts:
- added D12: BAT165, project_footprints:D_SOD-323, symbol Diode:B160-E3
Connections:
- net labels added: +5V, +5VP
- net labels removed: P3V3_HAT
- wire segments 87 -> 92
- no-connect marks 27 -> 28
Other:
- moved on the sheet: D10, D11

Commit message: Finally have the stackup
Parts:
- added R7, R9: 3.9K, project_footprints:R_0402, symbol Device:R
- R11, R29: footprint project_footprints:R_0603_1608Metric_Pad0.84x1.00mm_HandSolder -> project_footprints:R_0402; Alternate Part Number (none) -> RMCF0402FT10K0; Description (none) -> RES SMD 10K OHM 1% 1/10W 0402; MFR Yageo -> (none); MPN RC0402JR-0722RL -> (none); Manufacturer (none) -> Panasonic; Package (none) -> 0402; Part Number (none) -> ERJ-2RKF1002X; SPN 311-22JRCT-ND -> (none); SPR Digikey -> (none)
- R6, R8: footprint project_footprints:R_0603_1608Metric_Pad0.84x1.00mm_HandSolder -> project_footprints:R_0402; Alternate Part Number (none) -> CR0402-FX-3901GLF; Description (none) -> RES SMD 3.9K OHM 1% 1/10W 0402; MFR Yageo -> (none); MPN RC0402JR-0722RL -> (none); Manufacturer (none) -> Panasonic; Package (none) -> 0402; Part Number (none) -> RC0402FR-073K9L; SPN 311-22JRCT-ND -> (none); SPR Digikey -> (none)
Connections:
- net labels added: PI_SCL, PI_SDA
- wire segments 92 -> 108
- no-connect marks 28 -> 26
Changed lines of the file:
@@
 	1    0    0    -1
-$EndComp
-$Comp
-L Device:R R6
-U 1 1 58E17715
-P 2350 7400
-F 0 "R6" V 2430 7400 50  0000 C CNN
-F 1 "3.9K" V 2350 7400 50  0000 C CNN
-F 2 "project_footprints:R_0603_1608Metric_Pad0.84x1.00mm_HandSolder" V 2280 7400 50  0001 C CNN
-F 3 "" H 2350 7400 50  0001 C CNN
-F 4 "Yageo" H -13200 -6950 50  0001 C CNN "MFR"
-F 5 "RC0402JR-0722RL" H -13200 -6950 50  0001 C CNN "MPN"
-F 6 "Digikey" H -13200 -6950 50  0001 C CNN "SPR"
-F 7 "311-22JRCT-ND" H -13200 -6950 50  0001 C CNN "SPN"
-F 8 "" H -13200 -6950 50  0001 C CNN "SPURL"
-	1    2350 7400
-	0    1    1    0
-$EndComp
-$Comp
-L Device:R R8
-U 1 1 58E17720
-P 2350 7650
-F 0 "R8" V 2430 7650 50  0000 C CNN
-F 1 "3.9K" V 2350 7650 50  0000 C CNN
-F 2 "project_footprints:R_0603_1608Metric_Pad0.84x1.00mm_HandSolder" V 2280 7650 50  0001 C CNN
-F 3 "" H 2350 7650 50  0001 C CNN
-F 4 "Yageo" H -13200 -6700 50  0001 C CNN "MFR"
-F 5 "RC0402JR-0722RL" H -13200 -6700 50  0001 C CNN "MPN"
-F 6 "Digikey" H -13200 -6700 50  0001 C CNN "SPR"
-F 7 "311-22JRCT-ND" H -13200 -6700 50  0001 C CNN "SPN"
-F 8 "" H -13200 -6700 50  0001 C CNN "SPURL"
-	1    2350 7650
-	0    1    1    0
 $EndComp
 Wire Wire Line
@@
 	-1   0    0    1
 $EndComp
-$Comp
-L Device:R R29
-U 1 1 58E19E51
-P 1550 6250
-F 0 "R29" V 1630 6250 50  0000 C CNN
-F 1 "10K" V 1550 6250 50  0000 C CNN
-F 2 "project_footprints:R_0603_1608Metric_Pad0.84x1.00mm_HandSolder" V 1480 6250 50  0001 C CNN
-F 3 "" H 1550 6250 50  0001 C CNN
-F 4 "Yageo" H -14000 -8100 50  0001 C CNN "MFR"
-F 5 "RC0402JR-0722RL" H -14000 -8100 50  0001 C CNN "MPN"
-F 6 "Digikey" H -14000 -8100 50  0001 C CNN "SPR"
-F 7 "311-22JRCT-ND" H -14000 -8100 50  0001 C CNN "SPN"
-F 8 "" H -14000 -8100 50  0001 C CNN "SPURL"
-	1    1550 6250
-	-1   0    0    1
-$EndComp
 Wire Wire Line
 	2100 5350 2100 5450
@@
 Text Notes 3100 5250 0    60   ~ 0
 EEPROM WRITE ENABLE
-$Comp
-L Device:R R11
-U 1 1 58E22900
-P 1300 6100
-F 0 "R11" V 1380 6100 50  0000 C CNN
-F 1 "DNP" V 1300 6100 50  0000 C CNN
-F 2 "project_footprints:R_0603_1608Metric_Pad0.84x1.00mm_HandSolder" V 1230 6100 50  0001 C CNN
-F 3 "" H 1300 6100 50  0001 C CNN
-F 4 "Yageo" H -14250 -8250 50  0001 C CNN "MFR"
-F 5 "RC0402JR-0722RL" H -14250 -8250 50  0001 C CNN "MPN"
-F 6 "Digikey" H -14250 -8250 50  0001 C CNN "SPR"
-F 7 "311-22JRCT-ND" H -14250 -8250 50  0001 C CNN "SPN"
-F 8 "" H -14250 -8250 50  0001 C CNN "SPURL"
-	1    1300 6100
-	0    1    1    0
-$EndComp
 Text Notes 1550 7050 0    118  ~ 24
 Pullup Resistors
@@
 F8 "SWB_V2" O R 9150 3850 50
 F9 "SWB_V3" O R 9150 3950 50
+F10 "PI_SDA" I L 8150 2950 50
+F11 "PI_SCL" I L 8150 3050 50
 $EndSheet
 $Sheet
@@
 Wire Wire Line
 	9150 3950 10250 3950
-NoConn ~ 2000 2350
-NoConn ~ 2000 2450
 NoConn ~ 2000 2550
 NoConn ~ 2000 2750
@@
 	6600 8500 6600 8550
 Wire Wire Line
-	6600 8550 7950 8550
+	6600 8550 7350 8550
 Connection ~ 7950 8550
 NoConn ~ 2000 2250
@@
 Wire Wire Line
 	6600 8000 6600 8200
+Wire Wire Line
+	800  2350 1300 2350
+Wire Wire Line
+	800  2450 1500 2450
+Text Label 850  2450 0    60   ~ 0
+PI_SCL
+Text Label 850  2350 0    60   ~ 0
+PI_SDA
+$Comp
+L power:+3.3V #PWR?
+U 1 1 5BBDB670
+P 1400 1800
+AR Path="/5C1B036A/5BBDB670" Ref="#PWR?"  Part="1"
+AR Path="/5BBDB670" Ref="#PWR0104"  Part="1"
+F 0 "#PWR0104" H 1400 1650 50  0001 C CNN
+F 1 "+3.3V" H 1415 1973 50  0000 C CNN
+F 2 "" H 1400 1800 50  0001 C CNN
+F 3 "" H 1400 1800 50  0001 C CNN
+	1    1400 1800
+	1    0    0    -1
+$EndComp
+Wire Wire Line
+	1300 1900 1300 1850
+Wire Wire Line
+	1300 1850 1400 1850
+Wire Wire Line
+	1500 1850 1500 1900
+Wire Wire Line
+	1400 1800 1400 1850
+Connection ~ 1400 1850
+Wire Wire Line
+	1400 1850 1500 1850
+Wire Wire Line
+	1300 2200 1300 2350
+Connection ~ 1300 2350
+Wire Wire Line
+	1300 2350 2000 2350
+Wire Wire Line
+	1500 2200 1500 2450
+Connection ~ 1500 2450
+Wire Wire Line
+	1500 2450 2000 2450
+$Comp
+L Device:R R?
+U 1 1 5BC14805
+P 2350 7650
+AR Path="/5C1B036A/5BC14805" Ref="R?"  Part="1"
+AR Path="/5BC14805" Ref="R8"  Part="1"
+F 0 "R8" V 2450 7600 50  0000 L CNN
+F 1 "3.9K" V 2350 7550 50  0000 L CNN
+F 2 "project_footprints:R_0402" V 2280 7650 50  0001 C CNN
+F 3 "~" H 2350 7650 50  0001 C CNN
+F 4 "Panasonic" H 2350 7650 50  0001 C CNN "Manufacturer"
+F 5 "RC0402FR-073K9L" H 2350 7650 50  0001 C CNN "Part Number"
+F 6 "0402" H 2350 7650 50  0001 C CNN "Package"
+F 7 "RES SMD 3.9K OHM 1% 1/10W 0402" H 2350 7650 50  0001 C CNN "Description"
+F 8 "CR0402-FX-3901GLF" H 2350 7650 50  0001 C CNN "Alternate Part Number"
+	1    2350 7650
+	0    1    1    0
+$EndComp
+$Comp
+L Device:R R?
+U 1 1 5BC1795B
+P 2350 7400
+AR Path="/5C1B036A/5BC1795B" Ref="R?"  Part="1"
+AR Path="/5BC1795B" Ref="R6"  Part="1"
+F 0 "R6" V 2450 7350 50  0000 L CNN
+F 1 "3.9K" V 2350 7300 50  0000 L CNN
+F 2 "project_footprints:R_0402" V 2280 7400 50  0001 C CNN
+F 3 "~" H 2350 7400 50  0001 C CNN
+F 4 "Panasonic" H 2350 7400 50  0001 C CNN "Manufacturer"
+F 5 "RC0402FR-073K9L" H 2350 7400 50  0001 C CNN "Part Number"
+F 6 "0402" H 2350 7400 50  0001 C CNN "Package"
+F 7 "RES SMD 3.9K OHM 1% 1/10W 0402" H 2350 7400 50  0001 C CNN "Description"
+F 8 "CR0402-FX-3901GLF" H 2350 7400 50  0001 C CNN "Alternate Part Number"
+	1    2350 7400
+	0    1    1    0
+$EndComp
+$Comp
+L Device:R R?
+U 1 1 5BC17DA9
+P 1300 2050
+AR Path="/5C1B036A/5BC17DA9" Ref="R?"  Part="1"
+AR Path="/5BC17DA9" Ref="R7"  Part="1"
+F 0 "R7" V 1400 2000 50  0000 L CNN
+F 1 "3.9K" V 1300 1950 50  0000 L CNN
+F 2 "project_footprints:R_0402" V 1230 2050 50  0001 C CNN
+F 3 "~" H 1300 2050 50  0001 C CNN
+F 4 "Panasonic" H 1300 2050 50  0001 C CNN "Manufacturer"
+F 5 "RC0402FR-073K9L" H 1300 2050 50  0001 C CNN "Part Number"
+F 6 "0402" H 1300 2050 50  0001 C CNN "Package"
+F 7 "RES SMD 3.9K OHM 1% 1/10W 0402" H 1300 2050 50  0001 C CNN "Description"
+F 8 "CR0402-FX-3901GLF" H 1300 2050 50  0001 C CNN "Alternate Part Number"
+	1    1300 2050
+	-1   0    0    1
+$EndComp
+$Comp
+L Device:R R?
+U 1 1 5BC180DD
+P 1500 2050
+AR Path="/5C1B036A/5BC180DD" Ref="R?"  Part="1"
+AR Path="/5BC180DD" Ref="R9"  Part="1"
+F 0 "R9" V 1600 2000 50  0000 L CNN
+F 1 "3.9K" V 1500 1950 50  0000 L CNN
+F 2 "project_footprints:R_0402" V 1430 2050 50  0001 C CNN
+F 3 "~" H 1500 2050 50  0001 C CNN
+F 4 "Panasonic" H 1500 2050 50  0001 C CNN "Manufacturer"
+F 5 "RC0402FR-073K9L" H 1500 2050 50  0001 C CNN "Part Number"
+F 6 "0402" H 1500 2050 50  0001 C CNN "Package"
+F 7 "RES SMD 3.9K OHM 1% 1/10W 0402" H 1500 2050 50  0001 C CNN "Description"
+F 8 "CR0402-FX-3901GLF" H 1500 2050 50  0001 C CNN "Alternate Part Number"
+	1    1500 2050
+	-1   0    0    1
+$EndComp
+$Comp
+L Device:R R?
+U 1 1 5BC18658
+P 1550 6250
+AR Path="/5C1B036A/5BC18658" Ref="R?"  Part="1"
+AR Path="/5BC18658" Ref="R29"  Part="1"
+F 0 "R29" V 1650 6200 50  0000 L CNN
+F 1 "10K" V 1550 6200 50  0000 L CNN
+F 2 "project_footprints:R_0402" V 1480 6250 50  0001 C CNN
+F 3 "~" H 1550 6250 50  0001 C CNN
+F 4 "Panasonic" H 1550 6250 50  0001 C CNN "Manufacturer"
+F 5 "ERJ-2RKF1002X" H 1550 6250 50  0001 C CNN "Part Number"
+F 6 "0402" H 1550 6250 50  0001 C CNN "Package"
+F 7 "RES SMD 10K OHM 1% 1/10W 0402" H 1550 6250 50  0001 C CNN "Description"
+F 8 "RMCF0402FT10K0" H 1550 6250 50  0001 C CNN "Alternate Part Number"
+	1    1550 6250
+	-1   0    0    1
+$EndComp
+$Comp
+L Device:R R?
+U 1 1 5BC1B548
+P 1300 6100
+AR Path="/5C1B036A/5BC1B548" Ref="R?"  Part="1"
+AR Path="/5BC1B548" Ref="R11"  Part="1"
+F 0 "R11" V 1200 6050 50  0000 L CNN
+F 1 "DNP" V 1300 6000 50  0000 L CNN
+F 2 "project_footprints:R_0402" V 1230 6100 50  0001 C CNN
+F 3 "~" H 1300 6100 50  0001 C CNN
+F 4 "Panasonic" H 1300 6100 50  0001 C CNN "Manufacturer"
+F 5 "ERJ-2RKF1002X" H 1300 6100 50  0001 C CNN "Part Number"
+F 6 "0402" H 1300 6100 50  0001 C CNN "Package"
+F 7 "RES SMD 10K OHM 1% 1/10W 0402" H 1300 6100 50  0001 C CNN "Description"
+F 8 "RMCF0402FT10K0" H 1300 6100 50  0001 C CNN "Alternate Part Number"
+	1    1300 6100
+	0    -1   -1   0
+$EndComp
+Text Label 7650 2950 0    60   ~ 0
+PI_SDA
+Text Label 7650 3050 0    60   ~ 0
+PI_SCL
+Wire Wire Line
+	7550 2950 8150 2950
+Wire Wire Line
+	7550 3050 8150 3050
+$Comp
+L power:PWR_FLAG #FLG?
+U 1 1 5BE4BF9A
+P 7350 8500
+AR Path="/5C1B036A/5BE4BF9A" Ref="#FLG?"  Part="1"
+AR Path="/5BE4BF9A" Ref="#FLG0101"  Part="1"
+F 0 "#FLG0101" H 7350 8575 50  0001 C CNN
+F 1 "PWR_FLAG" H 7350 8674 50  0000 C CNN
+F 2 "" H 7350 8500 50  0001 C CNN
+F 3 "~" H 7350 8500 50  0001 C CNN
+	1    7350 8500
+	1    0    0    -1
+$EndComp
+Wire Wire Line
+	7350 8500 7350 8550
+Connection ~ 7350 8550
+Wire Wire Line
+	7350 8550 7950 8550
+$Comp
+L power:PWR_FLAG #FLG?
+U 1 1 5BE666CF
+P 6250 8200
+AR Path="/5C1B036A/5BE666CF" Ref="#FLG?"  Part="1"
+AR Path="/5BE666CF" Ref="#FLG0102"  Part="1"
+F 0 "#FLG0102" H 6250 8275 50  0001 C CNN
+F 1 "PWR_FLAG" H 6250 8374 50  0000 C CNN
+F 2 "" H 6250 8200 50  0001 C CNN
+F 3 "~" H 6250 8200 50  0001 C CNN
+	1    6250 8200
+	1    0    0    -1
+$EndComp
+Wire Wire Line
+	6250 8200 6600 8200
+Connection ~ 6600 8200
 $EndSCHEMATC

Commit message: I think the layout is ready for review
Connections:
- net labels added: P3V3_HAT
- wire segments 108 -> 110
- no-connect marks 26 -> 25

Commit message: Cleaned up BOM and added part numbers to the layout.
Parts:
- C3, C4: Manufacturer (none) -> Samsung
- J3: value 40HAT -> DNF; Alternate Part Number (none) -> SSW-120-01-G-D; Description (none) -> 2x20 0.1\" female header; Manufacturer (none) -> Samtec; Notes (none) -> available from Adafruit; Part Number (none) -> SSW-120-01-G-D
- J9: Alternate Part Number (none) -> M20-9990246; Description (none) -> CONN HEADER 2POS VERT T/H; Manufacturer (none) -> Amphenol; Part Number (none) -> 77311-118-02LF
- U2: Description (none) -> IC EEPROM 32K I2C 1MHZ 8SOIC; Manufacturer (none) -> ON Semiconductor; Package (none) -> SOIC-8; Part Number (none) -> CAT24C32WI-GT3
Changed lines of the file:
@@
 encoding utf-8
 Sheet 1 3
-Title "Raspberry Pi HAT"
+Title "Multi-Band Low Noise Amplifier"
 Date ""
 Rev "A"
-Comp ""
+Comp "SCH: 505-201"
 Comment1 ""
 Comment2 ""
@@
 P 2600 2250
 F 0 "J3" H 2950 2350 50  0000 C CNN
-F 1 "40HAT" H 2300 2350 50  0000 C CNN
+F 1 "DNF" H 2300 2350 50  0000 C CNN
 F 2 "project_footprints:PinSocket_2x20_P2.54mm_Vertical" H 2600 2450 50  0001 C CNN
-F 3 "" H 1900 2250 50  0000 C CNN
+F 3 "https://cdn-shop.adafruit.com/product-files/2243/12768.pdf" H 1900 2250 50  0001 C CNN
+F 4 "Samtec" H 2600 2250 50  0001 C CNN "Manufacturer"
+F 5 "SSW-120-01-G-D" H 2600 2250 50  0001 C CNN "Part Number"
+F 6 "2x20 0.1\" female header" H 2600 2250 50  0001 C CNN "Description"
+F 7 "available from Adafruit" H 2600 2250 50  0001 C CNN "Notes"
+F 8 "SSW-120-01-G-D" H 2600 2250 50  0001 C CNN "Alternate Part Number"
 	1    2600 2250
 	1    0    0    -1
@@
 F 2 "project_footprints:SOIC-8_3.9x4.9mm_P1.27mm" H 2100 5850 50  0001 C CNN
 F 3 "" H 2100 5850 50  0000 C CNN
+F 4 "ON Semiconductor" H 2100 5850 50  0001 C CNN "Manufacturer"
+F 5 "CAT24C32WI-GT3" H 2100 5850 50  0001 C CNN "Part Number"
+F 6 "SOIC-8" H 2100 5850 50  0001 C CNN "Package"
+F 7 "IC EEPROM 32K I2C 1MHZ 8SOIC" H 2100 5850 50  0001 C CNN "Description"
 	1    2100 5850
 	1    0    0    -1
@@
 F 2 "project_footprints:PinHeader_1x02_P2.54mm_Vertical" H 750 6100 50  0001 C CNN
 F 3 "" H 750 6100 50  0000 C CNN
+F 4 "Amphenol" H 750 6100 50  0001 C CNN "Manufacturer"
+F 5 "77311-118-02LF" H 750 6100 50  0001 C CNN "Part Number"
+F 6 "CONN HEADER 2POS VERT T/H" H 750 6100 50  0001 C CNN "Description"
+F 7 "M20-9990246" H 750 6100 50  0001 C CNN "Alternate Part Number"
 	1    750  6100
 	-1   0    0    1
@@
 F 7 "6.3V or greater" H 12450 6250 50  0001 C CNN "Notes"
 F 8 "GRM022R60J104ME15L" H 12450 6250 50  0001 C CNN "Alternate Part Number"
+F 9 "Samsung" H 0   0   50  0001 C CNN "Manufacturer"
 	1    12450 6250
 	1    0    0    -1
@@
 F 7 "6.3V or greater" H 12300 7650 50  0001 C CNN "Notes"
 F 8 "GRM022R60J104ME15L" H 12300 7650 50  0001 C CNN "Alternate Part Number"
+F 9 "Samsung" H 0   0   50  0001 C CNN "Manufacturer"
 	1    12300 7650
 	1    0    0    -1
